Commit message: Error in pepper.urdf.xacro file fixed, to spawn robot in Gazebo.

File: src/hrobot_description/urdf/pepper.urdf (robot description, URDF)
Before this commit: robot pepper_robot, 51 links, 50 joints
Links:
- link Head: geometry collision mesh filename=file:///media/mikelap/DATA2/Development/GithubRepos/hospita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 scale=0.1 0.1 0.1; visual mesh filename=file:///media/mikelap/DATA2/Development/GithubRepos/hospita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 scale=0.1 0.1 0.1
- link Hip: geometry collision mesh filename=file:///media/mikelap/DATA2/Development/GithubRepos/hospita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 scale=0.1 0.1 0.1; visual mesh filename=file:///media/mikelap/DATA2/Development/GithubRepos/hospita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 scale=0.1 0.1 0.1
- link LBicep: geometry collision mesh filename=file:///media/mikelap/DATA2/Development/GithubRepos/hospita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 scale=0.1 0.1 0.1; visual mesh filename=file:///media/mikelap/DATA2/Development/GithubRepos/hospita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 scale=0.1 0.1 0.1
- link LElbow: geometry collision mesh filename=file:///media/mikelap/DATA2/Development/GithubRepos/hospita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 scale=0.1 0.1 0.1; visual mesh filename=file:///media/mikelap/DATA2/Development/GithubRepos/hospita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 scale=0.1 0.1 0.1
- link LFinger11_link: geometry collision mesh filename=file:///media/mikelap/DATA2/Development/GithubRepos/hospita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 scale=0.1 0.1 0.1; visual mesh filename=file:///media/mikelap/DATA2/Development/GithubRepos/hospita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 scale=0.1 0.1 0.1
- link LFinger12_link: geometry collision mesh filename=file:///media/mikelap/DATA2/Development/GithubRepos/hospita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 scale=0.1 0.1 0.1; visual mesh filename=file:///media/mikelap/DATA2/Development/GithubRepos/hospita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 scale=0.1 0.1 0.1
- link LFinger13_link: geometry collision mesh filename=file:///media/mikelap/DATA2/Development/GithubRepos/hospita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 scale=0.1 0.1 0.1; visual mesh filename=file:///media/mikelap/DATA2/Development/GithubRepos/hospita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 scale=0.1 0.1 0.1
- link LFinger21_link: geometry collision mesh filename=file:///media/mikelap/DATA2/Development/GithubRepos/hospita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 scale=0.1 0.1 0.1; visual mesh filename=file:///media/mikelap/DATA2/Development/GithubRepos/hospita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 scale=0.1 0.1 0.1
- link LFinger22_link: geometry collision mesh filename=file:///media/mikelap/DATA2/Development/GithubRepos/hospita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 scale=0.1 0.1 0.1; visual mesh filename=file:///media/mikelap/DATA2/Development/GithubRepos/hospita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 scale=0.1 0.1 0.1
- link LFinger23_link: geometry collision mesh filename=file:///media/mikelap/DATA2/Development/GithubRepos/hospita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 scale=0.1 0.1 0.1; visual mesh filename=file:///media/mikelap/DATA2/Development/GithubRepos/hospita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 scale=0.1 0.1 0.1
- link LFinger31_link: geometry collision mesh filename=file:///media/mikelap/DATA2/Development/GithubRepos/hospita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 scale=0.1 0.1 0.1; visual mesh filename=file:///media/mikelap/DATA2/Development/GithubRepos/hospita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 scale=0.1 0.1 0.1
- link LFinger32_link: geometry collision mesh filename=file:///media/mikelap/DATA2/Development/GithubRepos/hospita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 scale=0.1 0.1 0.1; visual mesh filename=file:///media/mikelap/DATA2/Development/GithubRepos/hospita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 scale=0.1 0.1 0.1
- link LFinger33_link: geometry collision mesh filename=file:///media/mikelap/DATA2/Development/GithubRepos/hospita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 scale=0.1 0.1 0.1; visual mesh filename=file:///media/mikelap/DATA2/Development/GithubRepos/hospita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 scale=0.1 0.1 0.1
- link LFinger41_link: geometry collision mesh filename=file:///media/mikelap/DATA2/Development/GithubRepos/hospita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 scale=0.1 0.1 0.1; visual mesh filename=file:///media/mikelap/DATA2/Development/GithubRepos/hospita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 scale=0.1 0.1 0.1
- link LFinger42_link: geometry collision mesh filename=file:///media/mikelap/DATA2/Development/GithubRepos/hospita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 scale=0.1 0.1 0.1; visual mesh filename=file:///media/mikelap/DATA2/Development/GithubRepos/hospita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 scale=0.1 0.1 0.1
- link LFinger43_link: geometry collision mesh filename=file:///media/mikelap/DATA2/Development/GithubRepos/hospita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 scale=0.1 0.1 0.1; visual mesh filename=file:///media/mikelap/DATA2/Development/GithubRepos/hospita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 scale=0.1 0.1 0.1
- link LForeArm: geometry collision mesh filename=file:///media/mikelap/DATA2/Development/GithubRepos/hospita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 scale=0.1 0.1 0.1; visual mesh filename=file:///media/mikelap/DATA2/Development/GithubRepos/hospita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 scale=0.1 0.1 0.1
- link LShoulder: geometry collision mesh filename=file:///media/mikelap/DATA2/Development/GithubRepos/hospita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 scale=0.1 0.1 0.1; visual mesh filename=file:///media/mikelap/DATA2/Development/GithubRepos/hospita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 scale=0.1 0.1 0.1
- link LThumb1_link: geometry collision mesh filename=file:///media/mikelap/DATA2/Development/GithubRepos/hospita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 scale=0.1 0.1 0.1; visual mesh filename=file:///media/mikelap/DATA2/Development/GithubRepos/hospita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 scale=0.1 0.1 0.1
- link LThumb2_link: geometry collision mesh filename=file:///media/mikelap/DATA2/Development/GithubRepos/hospita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 scale=0.1 0.1 0.1; visual mesh filename=file:///media/mikelap/DATA2/Development/GithubRepos/hospita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 scale=0.1 0.1 0.1
- link Neck: geometry collision mesh filename=file:///media/mikelap/DATA2/Development/GithubRepos/hospita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 scale=0.1 0.1 0.1; visual mesh filename=file:///media/mikelap/DATA2/Development/GithubRepos/hospita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 scale=0.1 0.1 0.1
- link Pelvis: geometry collision mesh filename=file:///media/mikelap/DATA2/Development/GithubRepos/hospita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 scale=0.1 0.1 0.1; visual mesh filename=file:///media/mikelap/DATA2/Development/GithubRepos/hospita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 scale=0.1 0.1 0.1
- link RBicep: geometry collision mesh filename=file:///media/mikelap/DATA2/Development/GithubRepos/hospita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 scale=0.1 0.1 0.1; visual mesh filename=file:///media/mikelap/DATA2/Development/GithubRepos/hospita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 scale=0.1 0.1 0.1
- link RElbow: geometry collision mesh filename=file:///media/mikelap/DATA2/Development/GithubRepos/hospita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 scale=0.1 0.1 0.1; visual mesh filename=file:///media/mikelap/DATA2/Development/GithubRepos/hospita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 scale=0.1 0.1 0.1
- link RFinger11_link: geometry collision mesh filename=file:///media/mikelap/DATA2/Development/GithubRepos/hospita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 scale=0.1 0.1 0.1; visual mesh filename=file:///media/mikelap/DATA2/Development/GithubRepos/hospita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 scale=0.1 0.1 0.1
- link RFinger12_link: geometry collision mesh filename=file:///media/mikelap/DATA2/Development/GithubRepos/hospita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 scale=0.1 0.1 0.1; visual mesh filename=file:///media/mikelap/DATA2/Development/GithubRepos/hospita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 scale=0.1 0.1 0.1
- link RFinger13_link: geometry collision mesh filename=file:///media/mikelap/DATA2/Development/GithubRepos/hospita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 scale=0.1 0.1 0.1; visual mesh filename=file:///media/mikelap/DATA2/Development/GithubRepos/hospita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 scale=0.1 0.1 0.1
- link RFinger21_link: geometry collision mesh filename=file:///media/mikelap/DATA2/Development/GithubRepos/hospita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 scale=0.1 0.1 0.1; visual mesh filename=file:///media/mikelap/DATA2/Development/GithubRepos/hospita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 scale=0.1 0.1 0.1
- link RFinger22_link: geometry collision mesh filename=file:///media/mikelap/DATA2/Development/GithubRepos/hospita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 scale=0.1 0.1 0.1; visual mesh filename=file:///media/mikelap/DATA2/Development/GithubRepos/hospita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 scale=0.1 0.1 0.1
- link RFinger23_link: geometry collision mesh filename=file:///media/mikelap/DATA2/Development/GithubRepos/hospita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 scale=0.1 0.1 0.1; visual mesh filename=file:///media/mikelap/DATA2/Development/GithubRepos/hospita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 scale=0.1 0.1 0.1
- link RFinger31_link: geometry collision mesh filename=file:///media/mikelap/DATA2/Development/GithubRepos/hospita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 scale=0.1 0.1 0.1; visual mesh filename=file:///media/mikelap/DATA2/Development/GithubRepos/hospita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 scale=0.1 0.1 0.1
- link RFinger32_link: geometry collision mesh filename=file:///media/mikelap/DATA2/Development/GithubRepos/hospita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 scale=0.1 0.1 0.1; visual mesh filename=file:///media/mikelap/DATA2/Development/GithubRepos/hospita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 scale=0.1 0.1 0.1
- link RFinger33_link: geometry collision mesh filename=file:///media/mikelap/DATA2/Development/GithubRepos/hospita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 scale=0.1 0.1 0.1; visual mesh filename=file:///media/mikelap/DATA2/Development/GithubRepos/hospita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 scale=0.1 0.1 0.1
- link RFinger41_link: geometry collision mesh filename=file:///media/mikelap/DATA2/Development/GithubRepos/hospita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 scale=0.1 0.1 0.1; visual mesh filename=file:///media/mikelap/DATA2/Development/GithubRepos/hospita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 scale=0.1 0.1 0.1
- link RFinger42_link: geometry collision mesh filename=file:///media/mikelap/DATA2/Development/GithubRepos/hospita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 scale=0.1 0.1 0.1; visual mesh filename=file:///media/mikelap/DATA2/Development/GithubRepos/hospita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 scale=0.1 0.1 0.1
- link RFinger43_link: geometry collision mesh filename=file:///media/mikelap/DATA2/Development/GithubRepos/hospita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 scale=0.1 0.1 0.1; visual mesh filename=file:///media/mikelap/DATA2/Development/GithubRepos/hospita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 scale=0.1 0.1 0.1
- link RForeArm: geometry collision mesh filename=file:///media/mikelap/DATA2/Development/GithubRepos/hospita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 scale=0.1 0.1 0.1; visual mesh filename=file:///media/mikelap/DATA2/Development/GithubRepos/hospita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 scale=0.1 0.1 0.1
- link RShoulder: geometry collision mesh filename=file:///media/mikelap/DATA2/Development/GithubRepos/hospita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 scale=0.1 0.1 0.1; visual mesh filename=file:///media/mikelap/DATA2/Development/GithubRepos/hospita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 scale=0.1 0.1 0.1
- link RThumb1_link: geometry collision mesh filename=file:///media/mikelap/DATA2/Development/GithubRepos/hospita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 scale=0.1 0.1 0.1; visual mesh filename=file:///media/mikelap/DATA2/Development/GithubRepos/hospita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 scale=0.1 0.1 0.1
- link RThumb2_link: geometry collision mesh filename=file:///media/mikelap/DATA2/Development/GithubRepos/hospita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 scale=0.1 0.1 0.1; visual mesh filename=file:///media/mikelap/DATA2/Development/GithubRepos/hospita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 scale=0.1 0.1 0.1
- link Tibia: geometry collision mesh filename=file:///media/mikelap/DATA2/Development/GithubRepos/hospita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 scale=0.1 0.1 0.1; visual mesh filename=file:///media/mikelap/DATA2/Development/GithubRepos/hospita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 scale=0.1 0.1 0.1
- link WheelB_link: geometry collision mesh filename=file:///media/mikelap/DATA2/Development/GithubRepos/hospita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 scale=0.1 0.1 0.1; visual mesh filename=file:///media/mikelap/DATA2/Development/GithubRepos/hospita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 scale=0.1 0.1 0.1
- link WheelFL_link: geometry collision mesh filename=file:///media/mikelap/DATA2/Development/GithubRepos/hospita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 scale=0.1 0.1 0.1; visual mesh filename=file:///media/mikelap/DATA2/Development/GithubRepos/hospita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 scale=0.1 0.1 0.1
- link WheelFR_link: geometry collision mesh filename=file:///media/mikelap/DATA2/Development/GithubRepos/hospita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 scale=0.1 0.1 0.1; visual mesh filename=file:///media/mikelap/DATA2/Development/GithubRepos/hospita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 scale=0.1 0.1 0.1
- link l_wrist: geometry collision mesh filename=file:///media/mikelap/DATA2/Development/GithubRepos/hospita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 scale=0.1 0.1 0.1; visual mesh filename=file:///media/mikelap/DATA2/Development/GithubRepos/hospita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 scale=0.1 0.1 0.1
- link r_wrist: geometry collision mesh filename=file:///media/mikelap/DATA2/Development/GithubRepos/hospita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 scale=0.1 0.1 0.1; visual mesh filename=file:///media/mikelap/DATA2/Development/GithubRepos/hospita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 scale=0.1 0.1 0.1
- link torso: geometry collision mesh filename=file:///media/mikelap/DATA2/Development/GithubRepos/hospita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 scale=0.1 0.1 0.1; visual mesh filename=file:///media/mikelap/DATA2/Development/GithubRepos/hospita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 scale=0.1 0.1 0.1
