Commit message: Spawning error in Gazebo fixed (ros2_control still not implemented).

File: src/hrobot_description/urdf/pepper.urdf.xacro (robot description, xacro)
@@ -466,5 +466,5 @@
     <origin rpy="1.74402 1.04064 -0.0683394" xyz="0.074 -0.0309 0"/>
     <axis xyz="0 0 1.0"/>
-    <mimic joint="RHand" multiplier="0.872665" offset="0"/>
+    <!-- <mimic joint="RHand" multiplier="0.872665" offset="0"/> -->
   </joint>
   <link name="LFinger42_link">
@@ -491,5 +491,5 @@
     <origin rpy="0 0 -1.0472" xyz="0.018 0 0"/>
     <axis xyz="0 0 1.0"/>
-    <mimic joint="LHand" multiplier="0.872665" offset="0"/>
+    <!-- <mimic joint="LHand" multiplier="0.872665" offset="0"/> -->
   </joint>
   <link name="RFinger12_link">
@@ -516,5 +516,5 @@
     <origin rpy="0 0 -1.0472" xyz="0.018 0 0"/>
     <axis xyz="0 0 1.0"/>
-    <mimic joint="RHand" multiplier="0.872665" offset="0"/>
+    <!-- <mimic joint="RHand" multiplier="0.872665" offset="0"/> -->
   </joint>
   <link name="LFinger33_link">
@@ -541,5 +541,5 @@
     <origin rpy="0 0 -1.0472" xyz="0.018 0 0"/>
     <axis xyz="0 0 1.0"/>
-    <mimic joint="LHand" multiplier="0.872665" offset="0"/>
+    <!-- <mimic joint="LHand" multiplier="0.872665" offset="0"/> -->
   </joint>
   <link name="RFinger31_link">
@@ -566,5 +566,5 @@
     <origin rpy="1.67523 1.04483 0.029316" xyz="0.0833 -0.0123 0.004"/>
     <axis xyz="0 0 1.0"/>
-    <mimic joint="RHand" multiplier="0.872665" offset="0"/>
+    <!-- <mimic joint="RHand" multiplier="0.872665" offset="0"/> -->
   </joint>
   <link name="LFinger21_link">
@@ -591,5 +591,5 @@
     <origin rpy="1.5708 1.0472 -0.061086" xyz="0.0873 -0.0073 0.006"/>
     <axis xyz="0 0 1.0"/>
-    <mimic joint="LHand" multiplier="0.872665" offset="0"/>
+    <!-- <mimic joint="LHand" multiplier="0.872665" offset="0"/> -->
   </joint>
   <link name="RFinger32_link">
@@ -616,5 +616,5 @@
     <origin rpy="0 0 -1.0472" xyz="0.018 0 0"/>
     <axis xyz="0 0 1.0"/>
-    <mimic joint="RHand" multiplier="0.872665" offset="0"/>
+    <!-- <mimic joint="RHand" multiplier="0.872665" offset="0"/> -->
   </joint>
   <link name="LFinger13_link">
@@ -641,5 +641,5 @@
     <origin rpy="0 0 -1.0472" xyz="0.018 0 0"/>
     <axis xyz="0 0 1.0"/>
-    <mimic joint="LHand" multiplier="0.872665" offset="0"/>
+    <!-- <mimic joint="LHand" multiplier="0.872665" offset="0"/> -->
   </joint>
   <link name="LFinger32_link">
@@ -666,5 +666,5 @@
     <origin rpy="0 0 -1.0472" xyz="0.018 0 0"/>
     <axis xyz="0 0 1.0"/>
-    <mimic joint="LHand" multiplier="0.872665" offset="0"/>
+    <!-- <mimic joint="LHand" multiplier="0.872665" offset="0"/> -->
   </joint>
   <link name="LFinger11_link">
@@ -691,5 +691,5 @@
     <origin rpy="1.74402 1.04064 -0.0334335" xyz="0.0821 -0.0268 0.004"/>
     <axis xyz="0 0 1.0"/>
-    <mimic joint="LHand" multiplier="0.872665" offset="0"/>
+    <!-- <mimic joint="LHand" multiplier="0.872665" offset="0"/> -->
   </joint>
   <link name="RFinger22_link">
@@ -716,5 +716,5 @@
     <origin rpy="0 0 -1.0472" xyz="0.018 0 0"/>
     <axis xyz="0 0 1.0"/>
-    <mimic joint="RHand" multiplier="0.872665" offset="0"/>
+    <!-- <mimic joint="RHand" multiplier="0.872665" offset="0"/> -->
   </joint>
   <link name="RFinger13_link">
@@ -741,5 +741,5 @@
     <origin rpy="0 0 -1.0472" xyz="0.018 0 0"/>
     <axis xyz="0 0 1.0"/>
-    <mimic joint="RHand" multiplier="0.872665" offset="0"/>
+    <!-- <mimic joint="RHand" multiplier="0.872665" offset="0"/> -->
   </joint>
   <link name="LFinger22_link">
@@ -766,5 +766,5 @@
     <origin rpy="0 0 -1.0472" xyz="0.018 0 0"/>
     <axis xyz="0 0 1.0"/>
-    <mimic joint="LHand" multiplier="0.872665" offset="0"/>
+    <!-- <mimic joint="LHand" multiplier="0.872665" offset="0"/> -->
   </joint>
   <link name="RFinger21_link">
@@ -791,5 +791,5 @@
     <origin rpy="1.5708 1.0472 0.061086" xyz="0.0873 0.0073 0.006"/>
     <axis xyz="0 0 1.0"/>
-    <mimic joint="RHand" multiplier="0.872665" offset="0"/>
+    <!-- <mimic joint="RHand" multiplier="0.872665" offset="0"/> -->
   </joint>
   <link name="LFinger41_link">
@@ -816,5 +816,5 @@
     <origin rpy="1.39757 1.04064 0.0683394" xyz="0.074 0.0309 0"/>
     <axis xyz="0 0 1.0"/>
-    <mimic joint="LHand" multiplier="0.872665" offset="0"/>
+    <!-- <mimic joint="LHand" multiplier="0.872665" offset="0"/> -->
   </joint>
   <link name="LFinger12_link">
@@ -841,5 +841,5 @@
     <origin rpy="0 0 -1.0472" xyz="0.018 0 0"/>
     <axis xyz="0 0 1.0"/>
-    <mimic joint="LHand" multiplier="0.872665" offset="0"/>
+    <!-- <mimic joint="LHand" multiplier="0.872665" offset="0"/> -->
   </joint>
   <link name="RFinger23_link">
@@ -866,5 +866,5 @@
     <origin rpy="0 0 -1.0472" xyz="0.018 0 0"/>
     <axis xyz="0 0 1.0"/>
-    <mimic joint="RHand" multiplier="0.872665" offset="0"/>
+    <!-- <mimic joint="RHand" multiplier="0.872665" offset="0"/> -->
   </joint>
   <link name="RFinger11_link">
@@ -891,5 +891,5 @@
     <origin rpy="1.39757 1.04064 0.0334335" xyz="0.0821 0.0268 0.004"/>
     <axis xyz="0 0 1.0"/>
-    <mimic joint="RHand" multiplier="0.872665" offset="0"/>
+    <!-- <mimic joint="RHand" multiplier="0.872665" offset="0"/> -->
   </joint>
   <link name="LFinger23_link">
@@ -916,5 +916,5 @@
     <origin rpy="0 0 -1.0472" xyz="0.018 0 0"/>
     <axis xyz="0 0 1.0"/>
-    <mimic joint="LHand" multiplier="0.872665" offset="0"/>
+    <!-- <mimic joint="LHand" multiplier="0.872665" offset="0"/> -->
   </joint>
   <link name="LFinger43_link">
@@ -941,5 +941,5 @@
     <origin rpy="0 0 -1.0472" xyz="0.018 0 0"/>
     <axis xyz="0 0 1.0"/>
-    <mimic joint="LHand" multiplier="0.872665" offset="0"/>
+    <!-- <mimic joint="LHand" multiplier="0.872665" offset="0"/> -->
   </joint>
   <link name="RFinger43_link">
@@ -966,5 +966,5 @@
     <origin rpy="0 0 -1.0472" xyz="0.018 0 0"/>
     <axis xyz="0 0 1.0"/>
-    <mimic joint="RHand" multiplier="0.872665" offset="0"/>
+    <!-- <mimic joint="RHand" multiplier="0.872665" offset="0"/> -->
   </joint>
   <link name="RFinger42_link">
@@ -991,5 +991,5 @@
     <origin rpy="0 0 -1.0472" xyz="0.018 0 0"/>
     <axis xyz="0 0 1.0"/>
-    <mimic joint="RHand" multiplier="0.872665" offset="0"/>
+    <!-- <mimic joint="RHand" multiplier="0.872665" offset="0"/> -->
   </joint>
   <link name="LFinger31_link">
@@ -1016,5 +1016,5 @@
     <origin rpy="1.46636 1.04483 -0.029314" xyz="0.0833 0.0123 0.004"/>
     <axis xyz="0 0 1.0"/>
-    <mimic joint="LHand" multiplier="0.872665" offset="0"/>
+    <!-- <mimic joint="LHand" multiplier="0.872665" offset="0"/> -->
   </joint>
   <link name="RFinger33_link">
@@ -1041,5 +1041,5 @@
     <origin rpy="0 0 -1.0472" xyz="0.018 0 0"/>
     <axis xyz="0 0 1.0"/>
-    <mimic joint="RHand" multiplier="0.872665" offset="0"/>
+    <!-- <mimic joint="RHand" multiplier="0.872665" offset="0"/> -->
   </joint>
   <link name="LThumb1_link">
@@ -1066,5 +1066,5 @@
     <origin rpy="-1.95836 0.60626 0.533978" xyz="0.0482 -0.0357 -0.0199"/>
     <axis xyz="0 0 1.0"/>
-    <mimic joint="LHand" multiplier="0.872665" offset="0"/>
+    <!-- <mimic joint="LHand" multiplier="0.872665" offset="0"/> -->
   </joint>
   <link name="RThumb2_link">
@@ -1091,5 +1091,5 @@
     <origin rpy="0 0 -1.0472" xyz="0.022 0 0"/>
     <axis xyz="0 0 1.0"/>
-    <mimic joint="RHand" multiplier="0.872665" offset="0"/>
+    <!-- <mimic joint="RHand" multiplier="0.872665" offset="0"/> -->
   </joint>
   <link name="RThumb1_link">
@@ -1116,5 +1116,5 @@
     <origin rpy="-1.18323 0.60626 -0.533978" xyz="0.0482 0.0357 -0.0199"/>
     <axis xyz="0 0 1.0"/>
-    <mimic joint="RHand" multiplier="0.872665" offset="0"/>
+    <!-- <mimic joint="RHand" multiplier="0.872665" offset="0"/> -->
   </joint>
   <link name="LThumb2_link">
@@ -1141,5 +1141,5 @@
     <origin rpy="0 0 -1.0472" xyz="0.022 0 0"/>
     <axis xyz="0 0 1.0"/>
-    <mimic joint="LHand" multiplier="0.872665" offset="0"/>
+    <!-- <mimic joint="LHand" multiplier="0.872665" offset="0"/> -->
   </joint>
   <link name="WheelFL_link">

Commit message: mimic joints reactivated, because of the physics engine change from DART to Bullet ~ (ros2_control still not implemented).

File: src/hrobot_description/urdf/pepper.urdf.xacro (robot description, xacro)
@@ -466,5 +466,5 @@
     <origin rpy="1.74402 1.04064 -0.0683394" xyz="0.074 -0.0309 0"/>
     <axis xyz="0 0 1.0"/>
-    <!-- <mimic joint="RHand" multiplier="0.872665" offset="0"/> -->
+    <mimic joint="RHand" multiplier="0.872665" offset="0"/>
   </joint>
   <link name="LFinger42_link">
@@ -491,5 +491,5 @@
     <origin rpy="0 0 -1.0472" xyz="0.018 0 0"/>
     <axis xyz="0 0 1.0"/>
-    <!-- <mimic joint="LHand" multiplier="0.872665" offset="0"/> -->
+    <mimic joint="LHand" multiplier="0.872665" offset="0"/>
   </joint>
   <link name="RFinger12_link">
@@ -516,5 +516,5 @@
     <origin rpy="0 0 -1.0472" xyz="0.018 0 0"/>
     <axis xyz="0 0 1.0"/>
-    <!-- <mimic joint="RHand" multiplier="0.872665" offset="0"/> -->
+    <mimic joint="RHand" multiplier="0.872665" offset="0"/>
   </joint>
   <link name="LFinger33_link">
@@ -541,5 +541,5 @@
     <origin rpy="0 0 -1.0472" xyz="0.018 0 0"/>
     <axis xyz="0 0 1.0"/>
-    <!-- <mimic joint="LHand" multiplier="0.872665" offset="0"/> -->
+    <mimic joint="LHand" multiplier="0.872665" offset="0"/>
   </joint>
   <link name="RFinger31_link">
@@ -566,5 +566,5 @@
     <origin rpy="1.67523 1.04483 0.029316" xyz="0.0833 -0.0123 0.004"/>
     <axis xyz="0 0 1.0"/>
-    <!-- <mimic joint="RHand" multiplier="0.872665" offset="0"/> -->
+    <mimic joint="RHand" multiplier="0.872665" offset="0"/>
   </joint>
   <link name="LFinger21_link">
@@ -591,5 +591,5 @@
     <origin rpy="1.5708 1.0472 -0.061086" xyz="0.0873 -0.0073 0.006"/>
     <axis xyz="0 0 1.0"/>
-    <!-- <mimic joint="LHand" multiplier="0.872665" offset="0"/> -->
+    <mimic joint="LHand" multiplier="0.872665" offset="0"/>
   </joint>
   <link name="RFinger32_link">
@@ -616,5 +616,5 @@
     <origin rpy="0 0 -1.0472" xyz="0.018 0 0"/>
     <axis xyz="0 0 1.0"/>
-    <!-- <mimic joint="RHand" multiplier="0.872665" offset="0"/> -->
+    <mimic joint="RHand" multiplier="0.872665" offset="0"/>
   </joint>
   <link name="LFinger13_link">
@@ -641,5 +641,5 @@
     <origin rpy="0 0 -1.0472" xyz="0.018 0 0"/>
     <axis xyz="0 0 1.0"/>
-    <!-- <mimic joint="LHand" multiplier="0.872665" offset="0"/> -->
+    <mimic joint="LHand" multiplier="0.872665" offset="0"/>
   </joint>
   <link name="LFinger32_link">
@@ -666,5 +666,5 @@
     <origin rpy="0 0 -1.0472" xyz="0.018 0 0"/>
     <axis xyz="0 0 1.0"/>
-    <!-- <mimic joint="LHand" multiplier="0.872665" offset="0"/> -->
+    <mimic joint="LHand" multiplier="0.872665" offset="0"/>
   </joint>
   <link name="LFinger11_link">
@@ -691,5 +691,5 @@
     <origin rpy="1.74402 1.04064 -0.0334335" xyz="0.0821 -0.0268 0.004"/>
     <axis xyz="0 0 1.0"/>
-    <!-- <mimic joint="LHand" multiplier="0.872665" offset="0"/> -->
+    <mimic joint="LHand" multiplier="0.872665" offset="0"/>
   </joint>
   <link name="RFinger22_link">
@@ -716,5 +716,5 @@
     <origin rpy="0 0 -1.0472" xyz="0.018 0 0"/>
     <axis xyz="0 0 1.0"/>
-    <!-- <mimic joint="RHand" multiplier="0.872665" offset="0"/> -->
+    <mimic joint="RHand" multiplier="0.872665" offset="0"/>
   </joint>
   <link name="RFinger13_link">
@@ -741,5 +741,5 @@
     <origin rpy="0 0 -1.0472" xyz="0.018 0 0"/>
     <axis xyz="0 0 1.0"/>
-    <!-- <mimic joint="RHand" multiplier="0.872665" offset="0"/> -->
+    <mimic joint="RHand" multiplier="0.872665" offset="0"/>
   </joint>
   <link name="LFinger22_link">
@@ -766,5 +766,5 @@
     <origin rpy="0 0 -1.0472" xyz="0.018 0 0"/>
     <axis xyz="0 0 1.0"/>
-    <!-- <mimic joint="LHand" multiplier="0.872665" offset="0"/> -->
+    <mimic joint="LHand" multiplier="0.872665" offset="0"/>
   </joint>
   <link name="RFinger21_link">
@@ -791,5 +791,5 @@
     <origin rpy="1.5708 1.0472 0.061086" xyz="0.0873 0.0073 0.006"/>
     <axis xyz="0 0 1.0"/>
-    <!-- <mimic joint="RHand" multiplier="0.872665" offset="0"/> -->
+    <mimic joint="RHand" multiplier="0.872665" offset="0"/>
   </joint>
   <link name="LFinger41_link">
@@ -816,5 +816,5 @@
     <origin rpy="1.39757 1.04064 0.0683394" xyz="0.074 0.0309 0"/>
     <axis xyz="0 0 1.0"/>
-    <!-- <mimic joint="LHand" multiplier="0.872665" offset="0"/> -->
+    <mimic joint="LHand" multiplier="0.872665" offset="0"/>
   </joint>
   <link name="LFinger12_link">
@@ -841,5 +841,5 @@
     <origin rpy="0 0 -1.0472" xyz="0.018 0 0"/>
     <axis xyz="0 0 1.0"/>
-    <!-- <mimic joint="LHand" multiplier="0.872665" offset="0"/> -->
+    <mimic joint="LHand" multiplier="0.872665" offset="0"/>
   </joint>
   <link name="RFinger23_link">
@@ -866,5 +866,5 @@
     <origin rpy="0 0 -1.0472" xyz="0.018 0 0"/>
     <axis xyz="0 0 1.0"/>
-    <!-- <mimic joint="RHand" multiplier="0.872665" offset="0"/> -->
+    <mimic joint="RHand" multiplier="0.872665" offset="0"/>
   </joint>
   <link name="RFinger11_link">
@@ -891,5 +891,5 @@
     <origin rpy="1.39757 1.04064 0.0334335" xyz="0.0821 0.0268 0.004"/>
     <axis xyz="0 0 1.0"/>
-    <!-- <mimic joint="RHand" multiplier="0.872665" offset="0"/> -->
+    <mimic joint="RHand" multiplier="0.872665" offset="0"/>
   </joint>
   <link name="LFinger23_link">
@@ -916,5 +916,5 @@
     <origin rpy="0 0 -1.0472" xyz="0.018 0 0"/>
     <axis xyz="0 0 1.0"/>
-    <!-- <mimic joint="LHand" multiplier="0.872665" offset="0"/> -->
+    <mimic joint="LHand" multiplier="0.872665" offset="0"/>
   </joint>
   <link name="LFinger43_link">
@@ -941,5 +941,5 @@
     <origin rpy="0 0 -1.0472" xyz="0.018 0 0"/>
     <axis xyz="0 0 1.0"/>
-    <!-- <mimic joint="LHand" multiplier="0.872665" offset="0"/> -->
+    <mimic joint="LHand" multiplier="0.872665" offset="0"/>
   </joint>
   <link name="RFinger43_link">
@@ -966,5 +966,5 @@
     <origin rpy="0 0 -1.0472" xyz="0.018 0 0"/>
     <axis xyz="0 0 1.0"/>
-    <!-- <mimic joint="RHand" multiplier="0.872665" offset="0"/> -->
+    <mimic joint="RHand" multiplier="0.872665" offset="0"/>
   </joint>
   <link name="RFinger42_link">
@@ -991,5 +991,5 @@
     <origin rpy="0 0 -1.0472" xyz="0.018 0 0"/>
     <axis xyz="0 0 1.0"/>
-    <!-- <mimic joint="RHand" multiplier="0.872665" offset="0"/> -->
+    <mimic joint="RHand" multiplier="0.872665" offset="0"/>
   </joint>
   <link name="LFinger31_link">
@@ -1016,5 +1016,5 @@
     <origin rpy="1.46636 1.04483 -0.029314" xyz="0.0833 0.0123 0.004"/>
     <axis xyz="0 0 1.0"/>
-    <!-- <mimic joint="LHand" multiplier="0.872665" offset="0"/> -->
+    <mimic joint="LHand" multiplier="0.872665" offset="0"/>
   </joint>
   <link name="RFinger33_link">
@@ -1041,5 +1041,5 @@
     <origin rpy="0 0 -1.0472" xyz="0.018 0 0"/>
     <axis xyz="0 0 1.0"/>
-    <!-- <mimic joint="RHand" multiplier="0.872665" offset="0"/> -->
+    <mimic joint="RHand" multiplier="0.872665" offset="0"/>
   </joint>
   <link name="LThumb1_link">
@@ -1066,5 +1066,5 @@
     <origin rpy="-1.95836 0.60626 0.533978" xyz="0.0482 -0.0357 -0.0199"/>
     <axis xyz="0 0 1.0"/>
-    <!-- <mimic joint="LHand" multiplier="0.872665" offset="0"/> -->
+    <mimic joint="LHand" multiplier="0.872665" offset="0"/>
   </joint>
   <link name="RThumb2_link">
@@ -1091,5 +1091,5 @@
     <origin rpy="0 0 -1.0472" xyz="0.022 0 0"/>
     <axis xyz="0 0 1.0"/>
-    <!-- <mimic joint="RHand" multiplier="0.872665" offset="0"/> -->
+    <mimic joint="RHand" multiplier="0.872665" offset="0"/>
   </joint>
   <link name="RThumb1_link">
@@ -1116,5 +1116,5 @@
     <origin rpy="-1.18323 0.60626 -0.533978" xyz="0.0482 0.0357 -0.0199"/>
     <axis xyz="0 0 1.0"/>
-    <!-- <mimic joint="RHand" multiplier="0.872665" offset="0"/> -->
+    <mimic joint="RHand" multiplier="0.872665" offset="0"/>
   </joint>
   <link name="LThumb2_link">
@@ -1141,5 +1141,5 @@
     <origin rpy="0 0 -1.0472" xyz="0.022 0 0"/>
     <axis xyz="0 0 1.0"/>
-    <!-- <mimic joint="LHand" multiplier="0.872665" offset="0"/> -->
+    <mimic joint="LHand" multiplier="0.872665" offset="0"/>
   </joint>
   <link name="WheelFL_link">

Commit message: pepper.urdf.xacro modified (wheel orientation and position)

File: src/hrobot_description/urdf/pepper.urdf.xacro (robot description, xacro)
@@ -3,8 +3,8 @@
   <link name="base_footprint" />
   <link name="base_link"/>
-  <joint name="base_link_joint" type="fixed">
+  <joint name="base_joint" type="fixed">
     <parent link="base_footprint"/>
     <child link="base_link"/>
-    <origin rpy="0 0 0" xyz="0 0 0.1"/>
+    <origin rpy="0 0 0" xyz="0 0 -0.1"/>
   </joint>
   <joint name="HeadYaw" type="revolute">
@@ -138,4 +138,9 @@
     </inertial>
   </link>
+  <joint name="fixed_base" type="fixed">
+    <parent link="base_link"/>
+    <child link="Tibia"/>
+    <origin rpy="0 0 0" xyz="0 0 0.334"/>
+  </joint>
   <link name="torso">
     <visual>
@@ -1162,19 +1167,20 @@
     </inertial>
   </link>
-  <joint name="WheelFL" type="fixed">
+  <joint name="WheelFL" type="continuous">
     <parent link="Tibia"/>
     <child link="WheelFL_link"/>
-    <origin rpy="0 0 1.07517" xyz="0.09 0.155 -0.264"/>
-  </joint>
-  <link name="WheelB_link">
-    <visual>
-      <geometry>
-        <mesh filename="file://$(find hrobot_description)/meshes/WheelB.dae" scale="0.1 0.1 0.1"/>
-      </geometry>
-      <origin rpy="0 0 0" xyz="0 0 0"/>
-    </visual>
-    <collision>
-      <geometry>
-        <mesh filename="file://$(find hrobot_description)/meshes/WheelB_0.10.stl" scale="0.1 0.1 0.1"/>
+    <origin rpy="0 0 0" xyz="0.09 0.155 -0.264"/>
+    <axis xyz="0 1 0"/>
+  </joint>
+  <link name="WheelFR_link">
+    <visual>
+      <geometry>
+        <mesh filename="file://$(find hrobot_description)/meshes/WheelFR.dae" scale="0.1 0.1 0.1"/>
+      </geometry>
+      <origin rpy="0 0 0" xyz="0 0 0"/>
+    </visual>
+    <collision>
+      <geometry>
+        <mesh filename="file://$(find hrobot_description)/meshes/WheelFR_0.10.stl" scale="0.1 0.1 0.1"/>
       </geometry>
       <origin rpy="0 0 0" xyz="0 0 0"/>
@@ -1186,37 +1192,35 @@
     </inertial>
   </link>
-  <joint name="WheelB" type="fixed">
+  <joint name="WheelFR" type="continuous">
+    <parent link="Tibia"/>
+    <child link="WheelFR_link"/>
+    <origin rpy="0 0 0" xyz="0.09 -0.155 -0.264"/>
+    <axis xyz="0 1 0"/>
+  </joint>
+  <link name="WheelB_link">
+    <visual>
+      <geometry>
+        <mesh filename="file://$(find hrobot_description)/meshes/WheelB.dae" scale="0.1 0.1 0.1"/>
+      </geometry>
+      <origin rpy="0 0 0" xyz="0 0 0"/>
+    </visual>
+    <collision>
+      <geometry>
+        <mesh filename="file://$(find hrobot_description)/meshes/WheelB_0.10.stl" scale="0.1 0.1 0.1"/>
+      </geometry>
+      <origin rpy="0 0 0" xyz="0 0 0"/>
+    </collision>
+    <inertial>
+      <mass value="1.58028"/>
+      <inertia ixx="0.00299756" ixy="6.3068e-07" ixz="5.56903e-06" iyy="0.00303229" iyz="-9.0408e-07" izz="0.00296585"/>
+      <origin rpy="0 0 0" xyz="0 0 0"/>
+    </inertial>
+  </link>
+  <joint name="WheelB" type="continuous">
     <parent link="Tibia"/>
     <child link="WheelB_link"/>
-    <origin rpy="0 0 -3.14159" xyz="-0.17 0 -0.264"/>
-  </joint>
-  <link name="WheelFR_link">
-    <visual>
-      <geometry>
-        <mesh filename="file://$(find hrobot_description)/meshes/WheelFR.dae" scale="0.1 0.1 0.1"/>
-      </geometry>
-      <origin rpy="0 0 0" xyz="0 0 0"/>
-    </visual>
-    <collision>
-      <geometry>
-        <mesh filename="file://$(find hrobot_description)/meshes/WheelFR_0.10.stl" scale="0.1 0.1 0.1"/>
-      </geometry>
-      <origin rpy="0 0 0" xyz="0 0 0"/>
-    </collision>
-    <inertial>
-      <mass value="1.58028"/>
-      <inertia ixx="0.00299756" ixy="6.3068e-07" ixz="5.56903e-06" iyy="0.00303229" iyz="-9.0408e-07" izz="0.00296585"/>
-      <origin rpy="0 0 0" xyz="0 0 0"/>
-    </inertial>
-  </link>
-  <joint name="WheelFR" type="fixed">
-    <parent link="Tibia"/>
-    <child link="WheelFR_link"/>
-    <origin rpy="0 0 -1.07517" xyz="0.09 -0.155 -0.264"/>
-  </joint>
-  <joint name="fixed_base" type="fixed">
-    <parent link="base_link"/>
-    <child link="Tibia"/>
-    <origin rpy="0 0 0" xyz="0 0 0.234"/>
-  </joint>
+    <origin rpy="0 0 0" xyz="-0.17 0 -0.264"/>
+    <axis xyz="0 1 0"/>
+  </joint>
+  <xacro:include filename="$(find hrobot_description)/urdf/mobile_base_gazebo.xacro" />
 </robot>
