Commit message: Package for simulation in gazebo added.

File: src/hrobot_description/urdf/mobile_base_gazebo.xacro (robot description, xacro)
@@ -1,4 +1,8 @@
 <?xml version="1.0"?>
 <robot xmlns:xacro="http://www.ros.org/wiki/xacro">
+    <gazebo reference="WheelB_link">
+        <mu1 value="0.1" />
+        <mu2 value="0.1" />
+    </gazebo>
     <gazebo>
         <plugin filename="gz-sim-diff-drive-system" name="gz::sim::systems::DiffDrive">
@@ -7,6 +11,10 @@
             <frame_id>odom</frame_id>
             <child_frame_id>base_footprint</child_frame_id>
-            <wheel_separation>0.45</wheel_separation>
-            <wheel_radius>0.1</wheel_radius>
+            <wheel_separation>0.31</wheel_separation>
+            <wheel_radius>1.4</wheel_radius>
+        </plugin>
+    </gazebo>
+    <gazebo>
+        <plugin filename="gz-sim-joint-state-publisher-system" name="gz::sim::systems::JointStatePublisher">
         </plugin>
     </gazebo>

File: src/hrobot_description/urdf/pepper.urdf (robot description, URDF)
Before this commit: robot pepper_robot, 51 links, 50 joints
Joints:
- removed joint base_link_joint
- added joint base_joint: type fixed, parent base_footprint, child base_link, origin xyz=0 0 -0.1 rpy=0 0 0
- joint WheelB: origin xyz=-0.17 0 -0.264 rpy=0 0 -3.14159 -> xyz=-0.17 0 -0.264 rpy=0 0 0
- joint WheelFL: axis (none) -> 0 1 0; origin xyz=0.09 0.155 -0.264 rpy=0 0 1.07517 -> xyz=0.09 0.155 -0.264 rpy=0 0 0; type fixed -> continuous
- joint WheelFR: axis (none) -> 0 1 0; origin xyz=0.09 -0.155 -0.264 rpy=0 0 -1.07517 -> xyz=0.09 -0.155 -0.264 rpy=0 0 0; type fixed -> continuous
- joint fixed_base: origin xyz=0 0 0.234 rpy=0 0 0 -> xyz=0 0 0.334 rpy=0 0 0

File: src/hrobot_description/urdf/pepper.urdf.xacro (robot description, xacro)
@@ -1217,9 +1217,8 @@
     </inertial>
   </link>
-  <joint name="WheelB" type="continuous">
+  <joint name="WheelB" type="fixed">
     <parent link="Tibia"/>
     <child link="WheelB_link"/>
     <origin rpy="0 0 0" xyz="-0.17 0 -0.264"/>
-    <axis xyz="0 1 0"/>
   </joint>
   <xacro:include filename="$(find hrobot_description)/urdf/mobile_base_gazebo.xacro" />

Commit message: Gazebo plugins added and xacro files adapted.

File: src/hrobot_description/urdf/mobile_base_gazebo.xacro (robot description, xacro)
@@ -1,18 +1,211 @@
 <?xml version="1.0"?>
 <robot xmlns:xacro="http://www.ros.org/wiki/xacro">
+    <gazebo reference="Neck">
+        <mu1>0.2</mu1>
+        <mu2>0.2</mu2>
+    </gazebo>
+    <gazebo reference="Head">
+        <mu1>0.2</mu1>
+        <mu2>0.2</mu2>
+    </gazebo>
+    <gazebo reference="Hip">
+        <mu1>0.2</mu1>
+        <mu2>0.2</mu2>
+    </gazebo>
+    <gazebo reference="Pelvis">
+        <mu1>0.2</mu1>
+        <mu2>0.2</mu2>
+    </gazebo>
+    <gazebo reference="Tibia">
+        <mu1>0.2</mu1>
+        <mu2>0.2</mu2>
+    </gazebo>
+    <gazebo reference="torso">
+        <mu1>0.2</mu1>
+        <mu2>0.2</mu2>
+    </gazebo>
+    <gazebo reference="LShoulder">
+        <mu1>0.2</mu1>
+        <mu2>0.2</mu2>
+    </gazebo>
+    <gazebo reference="LBicep">
+        <mu1>0.2</mu1>
+        <mu2>0.2</mu2>
+    </gazebo>
+    <gazebo reference="LElbow">
+        <mu1>0.2</mu1>
+        <mu2>0.2</mu2>
+    </gazebo>
+    <gazebo reference="LForeArm">
+        <mu1>0.2</mu1>
+        <mu2>0.2</mu2>
+    </gazebo>
+    <gazebo reference="l_wrist">
+        <mu1>0.2</mu1>
+        <mu2>0.2</mu2>
+    </gazebo>
+    <gazebo reference="l_gripper">
+        <mu1>0.2</mu1>
+        <mu2>0.2</mu2>
+    </gazebo>
+    <gazebo reference="RShoulder">
+        <mu1>0.2</mu1>
+        <mu2>0.2</mu2>
+    </gazebo>
+    <gazebo reference="RBicep">
+        <mu1>0.2</mu1>
+        <mu2>0.2</mu2>
+    </gazebo>
+    <gazebo reference="RElbow">
+        <mu1>0.2</mu1>
+        <mu2>0.2</mu2>
+    </gazebo>
+    <gazebo reference="RForeArm">
+        <mu1>0.2</mu1>
+        <mu2>0.2</mu2>
+    </gazebo>
+    <gazebo reference="r_wrist">
+        <mu1>0.2</mu1>
+        <mu2>0.2</mu2>
+    </gazebo>
+    <gazebo reference="r_gripper">
+        <mu1>0.8</mu1>
+        <mu2>0.8</mu2>
+    </gazebo>
+    <gazebo reference="RFinger41_link">
+        <mu1>0.8</mu1>
+        <mu2>0.8</mu2>
+    </gazebo>
+    <gazebo reference="LFinger42_link">
+        <mu1>0.000002</mu1>
+        <mu2>0.000002</mu2>
+    </gazebo>
+    <gazebo reference="RFinger12_link">
+        <mu1>0.000002</mu1>
+        <mu2>0.000002</mu2>
+    </gazebo>
+    <gazebo reference="LFinger33_link">
+        <mu1>0.000002</mu1>
+        <mu2>0.000002</mu2>
+    </gazebo>
+    <gazebo reference="RFinger31_link">
+        <mu1>0.000002</mu1>
+        <mu2>0.000002</mu2>
+    </gazebo>
+    <gazebo reference="LFinger21_link">
+        <mu1>0.000002</mu1>
+        <mu2>0.000002</mu2>
+    </gazebo>
+    <gazebo reference="RFinger32_link">
+        <mu1>0.000002</mu1>
+        <mu2>0.000002</mu2>
+    </gazebo>
+    <gazebo reference="LFinger13_link">
+        <mu1>0.000002</mu1>
+        <mu2>0.000002</mu2>
+    </gazebo>
+    <gazebo reference="LFinger32_link">
+        <mu1>0.000002</mu1>
+        <mu2>0.000002</mu2>
+    </gazebo>
+    <gazebo reference="LFinger11_link">
+        <mu1>0.000002</mu1>
+        <mu2>0.000002</mu2>
+    </gazebo>
+    <gazebo reference="RFinger22_link">
+        <mu1>0.000002</mu1>
+        <mu2>0.000002</mu2>
+    </gazebo>
+    <gazebo reference="RFinger13_link">
+        <mu1>0.000002</mu1>
+        <mu2>0.000002</mu2>
+    </gazebo>
+    <gazebo reference="LFinger22_link">
+        <mu1>0.000002</mu1>
+        <mu2>0.000002</mu2>
+    </gazebo>
+    <gazebo reference="RFinger21_link">
+        <mu1>0.000002</mu1>
+        <mu2>0.000002</mu2>
+    </gazebo>
+    <gazebo reference="LFinger41_link">
+        <mu1>0.000002</mu1>
+        <mu2>0.000002</mu2>
+    </gazebo>
+    <gazebo reference="LFinger12_link">
+        <mu1>0.000002</mu1>
+        <mu2>0.000002</mu2>
+    </gazebo>
+    <gazebo reference="RFinger23_link">
+        <mu1>0.000002</mu1>
+        <mu2>0.000002</mu2>
+    </gazebo>
+    <gazebo reference="RFinger11_link">
+        <mu1>0.000002</mu1>
+        <mu2>0.000002</mu2>
+    </gazebo>
+    <gazebo reference="LFinger23_link">
+        <mu1>0.000002</mu1>
+        <mu2>0.000002</mu2>
+    </gazebo>
+    <gazebo reference="LFinger43_link">
+        <mu1>0.000002</mu1>
+        <mu2>0.000002</mu2>
+    </gazebo>
+    <gazebo reference="RFinger43_link">
+        <mu1>0.000002</mu1>
+        <mu2>0.000002</mu2>
+    </gazebo>
+    <gazebo reference="RFinger42_link">
+        <mu1>0.000002</mu1>
+        <mu2>0.000002</mu2>
+    </gazebo>
+    <gazebo reference="LFinger31_link">
+        <mu1>0.000002</mu1>
+        <mu2>0.000002</mu2>
+    </gazebo>
+    <gazebo reference="RFinger33_link">
+        <mu1>0.000002</mu1>
+        <mu2>0.000002</mu2>
+    </gazebo>
+    <gazebo reference="LThumb1_link">
+        <mu1>0.000002</mu1>
+        <mu2>0.000002</mu2>
+    </gazebo>
+    <gazebo reference="RThumb2_link">
+        <mu1>0.000002</mu1>
+        <mu2>0.000002</mu2>
+    </gazebo>
+    <gazebo reference="RThumb1_link">
+        <mu1>0.000002</mu1>
+        <mu2>0.000002</mu2>
+    </gazebo>
+    <gazebo reference="LThumb2_link">
+        <mu1>0.000002</mu1>
+        <mu2>0.000002</mu2>
+    </gazebo>
+    <gazebo reference="WheelFL_link">
+        <mu1>0.000002</mu1>
+        <mu2>0.000002</mu2>
+    </gazebo>
     <gazebo reference="WheelFR_link">
-        <mu1 value="0.8" />
-        <mu2 value="0.8" />
+        <mu1>0.000002</mu1>
+        <mu2>0.000002</mu2>
     </gazebo>
     <gazebo reference="WheelB_link">
-        <mu1 value="0.8" />
-        <mu2 value="0.8" />
-    </gazebo>
+        <mu1>0.000002</mu1>
+        <mu2>0.000002</mu2>
+    </gazebo>
+    <!-- Hardware interfaces -->
     <gazebo>
+        <!-- Diff drive -->
         <plugin filename="gz-sim-diff-drive-system" name="gz::sim::systems::DiffDrive">
             <left_joint>WheelFL</left_joint>
             <right_joint>WheelFR</right_joint>
             <frame_id>odom</frame_id>
+            <odom_topic>odom</odom_topic>
             <child_frame_id>base_footprint</child_frame_id>
+            <topic>cmd_vel</topic>
+            <tf_topic>/tf</tf_topic>
             <wheel_separation>0.31</wheel_separation>
             <wheel_radius>0.08</wheel_radius>
@@ -22,7 +215,9 @@
             <max_acceleration>10</max_acceleration>
         </plugin>
-    </gazebo>
-    <gazebo>
+        <!-- Joint state publisher -->
         <plugin filename="gz-sim-joint-state-publisher-system" name="gz::sim::systems::JointStatePublisher">
+            <topic>joint_states</topic>
+            <joint_name>WheelFL</joint_name>
+            <joint_name>WheelFR</joint_name>
         </plugin>
     </gazebo>

File: src/hrobot_description/urdf/pepper_robot.urdf.xacro (robot description, xacro)
@@ -1,4 +1,5 @@
 <?xml version="1.0"?>
 <robot name="pepper_robot" xmlns:xacro="http://www.ros.org/wiki/xacro">
+  <xacro:include filename="$(find hrobot_description)/urdf/mobile_base_gazebo.xacro" />
   <link name="base_footprint" />
   <link name="base_link"/>
@@ -1217,9 +1218,9 @@
     </inertial>
   </link>
-  <joint name="WheelB" type="fixed">
+  <joint name="WheelB" type="continuous">
     <parent link="Tibia"/>
     <child link="WheelB_link"/>
     <origin rpy="0 0 0" xyz="-0.17 0 -0.264"/>
-  </joint>
-  <xacro:include filename="$(find hrobot_description)/urdf/mobile_base_gazebo.xacro" />
+    <axis xyz="0 1 0"/>
+  </joint>
 </robot>

File: src/hrobot_description/urdf/pepper_robot_fixed.urdf.xacro (robot description, xacro)
@@ -1,4 +1,5 @@
 <?xml version="1.0"?>
 <robot name="pepper_robot" xmlns:xacro="http://www.ros.org/wiki/xacro">
+  <xacro:include filename="$(find hrobot_description)/urdf/mobile_base_gazebo.xacro" />
   <link name="base_footprint" />
   <link name="base_link"/>
