Commit message: Xacro file modified to exclude mimic joints (currently deactivated)

File: src/hrobot_description/urdf/pepper_robot.urdf.xacro (robot description, xacro)
@@ -468,10 +468,8 @@
     </inertial>
   </link>
-  <joint name="RFinger41" type="continuous">
+  <joint name="RFinger41" type="fixed">
     <parent link="r_wrist"/>
     <child link="RFinger41_link"/>
     <origin rpy="1.74402 1.04064 -0.0683394" xyz="0.074 -0.0309 0"/>
-    <axis xyz="0 0 1.0"/>
-    <mimic joint="RHand" multiplier="0.872665" offset="0"/>
   </joint>
   <link name="LFinger42_link">
@@ -493,10 +491,8 @@
     </inertial>
   </link>
-  <joint name="LFinger42" type="continuous">
+  <joint name="LFinger42" type="fixed">
     <parent link="LFinger41_link"/>
     <child link="LFinger42_link"/>
     <origin rpy="0 0 -1.0472" xyz="0.018 0 0"/>
-    <axis xyz="0 0 1.0"/>
-    <mimic joint="LHand" multiplier="0.872665" offset="0"/>
   </joint>
   <link name="RFinger12_link">
@@ -518,10 +514,8 @@
     </inertial>
   </link>
-  <joint name="RFinger12" type="continuous">
+  <joint name="RFinger12" type="fixed">
     <parent link="RFinger11_link"/>
     <child link="RFinger12_link"/>
     <origin rpy="0 0 -1.0472" xyz="0.018 0 0"/>
-    <axis xyz="0 0 1.0"/>
-    <mimic joint="RHand" multiplier="0.872665" offset="0"/>
   </joint>
   <link name="LFinger33_link">
@@ -543,10 +537,8 @@
     </inertial>
   </link>
-  <joint name="LFinger33" type="continuous">
+  <joint name="LFinger33" type="fixed">
     <parent link="LFinger32_link"/>
     <child link="LFinger33_link"/>
     <origin rpy="0 0 -1.0472" xyz="0.018 0 0"/>
-    <axis xyz="0 0 1.0"/>
-    <mimic joint="LHand" multiplier="0.872665" offset="0"/>
   </joint>
   <link name="RFinger31_link">
@@ -568,10 +560,8 @@
     </inertial>
   </link>
-  <joint name="RFinger31" type="continuous">
+  <joint name="RFinger31" type="fixed">
     <parent link="r_wrist"/>
     <child link="RFinger31_link"/>
     <origin rpy="1.67523 1.04483 0.029316" xyz="0.0833 -0.0123 0.004"/>
-    <axis xyz="0 0 1.0"/>
-    <mimic joint="RHand" multiplier="0.872665" offset="0"/>
   </joint>
   <link name="LFinger21_link">
@@ -593,10 +583,8 @@
     </inertial>
   </link>
-  <joint name="LFinger21" type="continuous">
+  <joint name="LFinger21" type="fixed">
     <parent link="l_wrist"/>
     <child link="LFinger21_link"/>
     <origin rpy="1.5708 1.0472 -0.061086" xyz="0.0873 -0.0073 0.006"/>
-    <axis xyz="0 0 1.0"/>
-    <mimic joint="LHand" multiplier="0.872665" offset="0"/>
   </joint>
   <link name="RFinger32_link">
@@ -618,10 +606,8 @@
     </inertial>
   </link>
-  <joint name="RFinger32" type="continuous">
+  <joint name="RFinger32" type="fixed">
     <parent link="RFinger31_link"/>
     <child link="RFinger32_link"/>
     <origin rpy="0 0 -1.0472" xyz="0.018 0 0"/>
-    <axis xyz="0 0 1.0"/>
-    <mimic joint="RHand" multiplier="0.872665" offset="0"/>
   </joint>
   <link name="LFinger13_link">
@@ -643,10 +629,8 @@
     </inertial>
   </link>
-  <joint name="LFinger13" type="continuous">
+  <joint name="LFinger13" type="fixed">
     <parent link="LFinger12_link"/>
     <child link="LFinger13_link"/>
     <origin rpy="0 0 -1.0472" xyz="0.018 0 0"/>
-    <axis xyz="0 0 1.0"/>
-    <mimic joint="LHand" multiplier="0.872665" offset="0"/>
   </joint>
   <link name="LFinger32_link">
@@ -668,10 +652,8 @@
     </inertial>
   </link>
-  <joint name="LFinger32" type="continuous">
+  <joint name="LFinger32" type="fixed">
     <parent link="LFinger31_link"/>
     <child link="LFinger32_link"/>
     <origin rpy="0 0 -1.0472" xyz="0.018 0 0"/>
-    <axis xyz="0 0 1.0"/>
-    <mimic joint="LHand" multiplier="0.872665" offset="0"/>
   </joint>
   <link name="LFinger11_link">
@@ -693,10 +675,8 @@
     </inertial>
   </link>
-  <joint name="LFinger11" type="continuous">
+  <joint name="LFinger11" type="fixed">
     <parent link="l_wrist"/>
     <child link="LFinger11_link"/>
     <origin rpy="1.74402 1.04064 -0.0334335" xyz="0.0821 -0.0268 0.004"/>
-    <axis xyz="0 0 1.0"/>
-    <mimic joint="LHand" multiplier="0.872665" offset="0"/>
   </joint>
   <link name="RFinger22_link">
@@ -718,10 +698,8 @@
     </inertial>
   </link>
-  <joint name="RFinger22" type="continuous">
+  <joint name="RFinger22" type="fixed">
     <parent link="RFinger21_link"/>
     <child link="RFinger22_link"/>
     <origin rpy="0 0 -1.0472" xyz="0.018 0 0"/>
-    <axis xyz="0 0 1.0"/>
-    <mimic joint="RHand" multiplier="0.872665" offset="0"/>
   </joint>
   <link name="RFinger13_link">
@@ -743,10 +721,8 @@
     </inertial>
   </link>
-  <joint name="RFinger13" type="continuous">
+  <joint name="RFinger13" type="fixed">
     <parent link="RFinger12_link"/>
     <child link="RFinger13_link"/>
     <origin rpy="0 0 -1.0472" xyz="0.018 0 0"/>
-    <axis xyz="0 0 1.0"/>
-    <mimic joint="RHand" multiplier="0.872665" offset="0"/>
   </joint>
   <link name="LFinger22_link">
@@ -768,10 +744,8 @@
     </inertial>
   </link>
-  <joint name="LFinger22" type="continuous">
+  <joint name="LFinger22" type="fixed">
     <parent link="LFinger21_link"/>
     <child link="LFinger22_link"/>
     <origin rpy="0 0 -1.0472" xyz="0.018 0 0"/>
-    <axis xyz="0 0 1.0"/>
-    <mimic joint="LHand" multiplier="0.872665" offset="0"/>
   </joint>
   <link name="RFinger21_link">
@@ -793,10 +767,8 @@
     </inertial>
   </link>
-  <joint name="RFinger21" type="continuous">
+  <joint name="RFinger21" type="fixed">
     <parent link="r_wrist"/>
     <child link="RFinger21_link"/>
     <origin rpy="1.5708 1.0472 0.061086" xyz="0.0873 0.0073 0.006"/>
-    <axis xyz="0 0 1.0"/>
-    <mimic joint="RHand" multiplier="0.872665" offset="0"/>
   </joint>
   <link name="LFinger41_link">
@@ -818,10 +790,8 @@
     </inertial>
   </link>
-  <joint name="LFinger41" type="continuous">
+  <joint name="LFinger41" type="fixed">
     <parent link="l_wrist"/>
     <child link="LFinger41_link"/>
     <origin rpy="1.39757 1.04064 0.0683394" xyz="0.074 0.0309 0"/>
-    <axis xyz="0 0 1.0"/>
-    <mimic joint="LHand" multiplier="0.872665" offset="0"/>
   </joint>
   <link name="LFinger12_link">
@@ -843,10 +813,8 @@
     </inertial>
   </link>
-  <joint name="LFinger12" type="continuous">
+  <joint name="LFinger12" type="fixed">
     <parent link="LFinger11_link"/>
     <child link="LFinger12_link"/>
     <origin rpy="0 0 -1.0472" xyz="0.018 0 0"/>
-    <axis xyz="0 0 1.0"/>
-    <mimic joint="LHand" multiplier="0.872665" offset="0"/>
   </joint>
   <link name="RFinger23_link">
@@ -868,10 +836,8 @@
     </inertial>
   </link>
-  <joint name="RFinger23" type="continuous">
+  <joint name="RFinger23" type="fixed">
     <parent link="RFinger22_link"/>
     <child link="RFinger23_link"/>
     <origin rpy="0 0 -1.0472" xyz="0.018 0 0"/>
-    <axis xyz="0 0 1.0"/>
-    <mimic joint="RHand" multiplier="0.872665" offset="0"/>
   </joint>
   <link name="RFinger11_link">
@@ -893,10 +859,8 @@
     </inertial>
   </link>
-  <joint name="RFinger11" type="continuous">
+  <joint name="RFinger11" type="fixed">
     <parent link="r_wrist"/>
     <child link="RFinger11_link"/>
     <origin rpy="1.39757 1.04064 0.0334335" xyz="0.0821 0.0268 0.004"/>
-    <axis xyz="0 0 1.0"/>
-    <mimic joint="RHand" multiplier="0.872665" offset="0"/>
   </joint>
   <link name="LFinger23_link">
@@ -918,10 +882,8 @@
     </inertial>
   </link>
-  <joint name="LFinger23" type="continuous">
+  <joint name="LFinger23" type="fixed">
     <parent link="LFinger22_link"/>
     <child link="LFinger23_link"/>
     <origin rpy="0 0 -1.0472" xyz="0.018 0 0"/>
-    <axis xyz="0 0 1.0"/>
-    <mimic joint="LHand" multiplier="0.872665" offset="0"/>
   </joint>
   <link name="LFinger43_link">
@@ -943,10 +905,8 @@
     </inertial>
   </link>
-  <joint name="LFinger43" type="continuous">
+  <joint name="LFinger43" type="fixed">
     <parent link="LFinger42_link"/>
     <child link="LFinger43_link"/>
     <origin rpy="0 0 -1.0472" xyz="0.018 0 0"/>
-    <axis xyz="0 0 1.0"/>
-    <mimic joint="LHand" multiplier="0.872665" offset="0"/>
   </joint>
   <link name="RFinger43_link">
@@ -968,10 +928,8 @@
     </inertial>
   </link>
-  <joint name="RFinger43" type="continuous">
+  <joint name="RFinger43" type="fixed">
     <parent link="RFinger42_link"/>
     <child link="RFinger43_link"/>
     <origin rpy="0 0 -1.0472" xyz="0.018 0 0"/>
-    <axis xyz="0 0 1.0"/>
-    <mimic joint="RHand" multiplier="0.872665" offset="0"/>
   </joint>
   <link name="RFinger42_link">
@@ -993,10 +951,8 @@
     </inertial>
   </link>
-  <joint name="RFinger42" type="continuous">
+  <joint name="RFinger42" type="fixed">
     <parent link="RFinger41_link"/>
     <child link="RFinger42_link"/>
     <origin rpy="0 0 -1.0472" xyz="0.018 0 0"/>
-    <axis xyz="0 0 1.0"/>
-    <mimic joint="RHand" multiplier="0.872665" offset="0"/>
   </joint>
   <link name="LFinger31_link">
@@ -1018,10 +974,8 @@
     </inertial>
   </link>
-  <joint name="LFinger31" type="continuous">
+  <joint name="LFinger31" type="fixed">
     <parent link="l_wrist"/>
     <child link="LFinger31_link"/>
     <origin rpy="1.46636 1.04483 -0.029314" xyz="0.0833 0.0123 0.004"/>
-    <axis xyz="0 0 1.0"/>
-    <mimic joint="LHand" multiplier="0.872665" offset="0"/>
   </joint>
   <link name="RFinger33_link">
@@ -1043,10 +997,8 @@
     </inertial>
   </link>
-  <joint name="RFinger33" type="continuous">
+  <joint name="RFinger33" type="fixed">
     <parent link="RFinger32_link"/>
     <child link="RFinger33_link"/>
     <origin rpy="0 0 -1.0472" xyz="0.018 0 0"/>
-    <axis xyz="0 0 1.0"/>
-    <mimic joint="RHand" multiplier="0.872665" offset="0"/>
   </joint>
   <link name="LThumb1_link">
@@ -1068,10 +1020,8 @@
     </inertial>
   </link>
-  <joint name="LThumb1" type="continuous">
+  <joint name="LThumb1" type="fixed">
     <parent link="l_wrist"/>
     <child link="LThumb1_link"/>
     <origin rpy="-1.95836 0.60626 0.533978" xyz="0.0482 -0.0357 -0.0199"/>
-    <axis xyz="0 0 1.0"/>
-    <mimic joint="LHand" multiplier="0.872665" offset="0"/>
   </joint>
   <link name="RThumb2_link">
@@ -1093,10 +1043,8 @@
     </inertial>
   </link>
-  <joint name="RThumb2" type="continuous">
+  <joint name="RThumb2" type="fixed">
     <parent link="RThumb1_link"/>
     <child link="RThumb2_link"/>
     <origin rpy="0 0 -1.0472" xyz="0.022 0 0"/>
-    <axis xyz="0 0 1.0"/>
-    <mimic joint="RHand" multiplier="0.872665" offset="0"/>
   </joint>
   <link name="RThumb1_link">
@@ -1118,10 +1066,8 @@
     </inertial>
   </link>
-  <joint name="RThumb1" type="continuous">
+  <joint name="RThumb1" type="fixed">
     <parent link="r_wrist"/>
     <child link="RThumb1_link"/>
     <origin rpy="-1.18323 0.60626 -0.533978" xyz="0.0482 0.0357 -0.0199"/>
-    <axis xyz="0 0 1.0"/>
-    <mimic joint="RHand" multiplier="0.872665" offset="0"/>
   </joint>
   <link name="LThumb2_link">
@@ -1143,10 +1089,8 @@
     </inertial>
   </link>
-  <joint name="LThumb2" type="continuous">
+  <joint name="LThumb2" type="fixed">
     <parent link="LThumb1_link"/>
     <child link="LThumb2_link"/>
     <origin rpy="0 0 -1.0472" xyz="0.022 0 0"/>
-    <axis xyz="0 0 1.0"/>
-    <mimic joint="LHand" multiplier="0.872665" offset="0"/>
   </joint>
   <link name="WheelFL_link">

File: src/hrobot_description/urdf/pepper_robot_fixed.urdf.xacro (robot description, xacro)
@@ -1,5 +1,4 @@
 <?xml version="1.0"?>
 <robot name="pepper_robot" xmlns:xacro="http://www.ros.org/wiki/xacro">
-  <xacro:include filename="$(find hrobot_description)/urdf/mobile_base_gazebo.xacro" />
   <link name="base_footprint" />
   <link name="base_link"/>
@@ -1134,4 +1133,3 @@
     <axis xyz="0 1 0"/>
   </joint>
-  <xacro:include filename="$(find hrobot_description)/urdf/mobile_base_gazebo.xacro" />
 </robot>

File: src/hrobot_kinematics/robot/hrobot_ros2_control.xacro (robot description, xacro)
@@ -175,5 +175,5 @@
             <state_interface name="effort"/>
         </joint>
-        <joint name="LFinger42">
+        <!-- <joint name="LFinger42">
             <command_interface name="velocity">
                 <param name="min">-1</param>
@@ -300,5 +300,5 @@
             <state_interface name="velocity"/>
             <state_interface name="effort"/>
-        </joint>
+        </joint> -->
         <!-- Right hand -->
         <joint name="RHand">
@@ -311,5 +311,5 @@
             <state_interface name="effort"/>
         </joint>
-        <joint name="RFinger41">
+        <!-- <joint name="RFinger41">
             <command_interface name="velocity">
                 <param name="min">-1</param>
@@ -436,5 +436,5 @@
             <state_interface name="velocity"/>
             <state_interface name="effort"/>
-        </joint>
+        </joint> -->
     </ros2_control>
     </robot>
