Commit message: ROS2 control joint management and settings updated

File: src/hrobot_description/urdf/gazebo_sim_ros2_control.urdf.xacro (robot description, xacro)
@@ -1,200 +1,4 @@
 <?xml version="1.0"?>
 <robot xmlns:xacro="http://www.ros.org/wiki/xacro">
-    <gazebo reference="Neck">
-        <mu1>0.2</mu1>
-        <mu2>0.2</mu2>
-    </gazebo>
-    <gazebo reference="Head">
-        <mu1>0.2</mu1>
-        <mu2>0.2</mu2>
-    </gazebo>
-    <gazebo reference="Hip">
-        <mu1>0.2</mu1>
-        <mu2>0.2</mu2>
-    </gazebo>
-    <gazebo reference="Pelvis">
-        <mu1>0.2</mu1>
-        <mu2>0.2</mu2>
-    </gazebo>
-    <gazebo reference="Tibia">
-        <mu1>0.2</mu1>
-        <mu2>0.2</mu2>
-    </gazebo>
-    <gazebo reference="torso">
-        <mu1>0.2</mu1>
-        <mu2>0.2</mu2>
-    </gazebo>
-    <gazebo reference="LShoulder">
-        <mu1>0.2</mu1>
-        <mu2>0.2</mu2>
-    </gazebo>
-    <gazebo reference="LBicep">
-        <mu1>0.2</mu1>
-        <mu2>0.2</mu2>
-    </gazebo>
-    <gazebo reference="LElbow">
-        <mu1>0.2</mu1>
-        <mu2>0.2</mu2>
-    </gazebo>
-    <gazebo reference="LForeArm">
-        <mu1>0.2</mu1>
-        <mu2>0.2</mu2>
-    </gazebo>
-    <gazebo reference="l_wrist">
-        <mu1>0.2</mu1>
-        <mu2>0.2</mu2>
-    </gazebo>
-    <gazebo reference="l_gripper">
-        <mu1>0.2</mu1>
-        <mu2>0.2</mu2>
-    </gazebo>
-    <gazebo reference="RShoulder">
-        <mu1>0.2</mu1>
-        <mu2>0.2</mu2>
-    </gazebo>
-    <gazebo reference="RBicep">
-        <mu1>0.2</mu1>
-        <mu2>0.2</mu2>
-    </gazebo>
-    <gazebo reference="RElbow">
-        <mu1>0.2</mu1>
-        <mu2>0.2</mu2>
-    </gazebo>
-    <gazebo reference="RForeArm">
-        <mu1>0.2</mu1>
-        <mu2>0.2</mu2>
-    </gazebo>
-    <gazebo reference="r_wrist">
-        <mu1>0.2</mu1>
-        <mu2>0.2</mu2>
-    </gazebo>
-    <gazebo reference="r_gripper">
-        <mu1>0.8</mu1>
-        <mu2>0.8</mu2>
-    </gazebo>
-    <gazebo reference="RFinger41_link">
-        <mu1>0.8</mu1>
-        <mu2>0.8</mu2>
-    </gazebo>
-    <gazebo reference="LFinger42_link">
-        <mu1>0.000002</mu1>
-        <mu2>0.000002</mu2>
-    </gazebo>
-    <gazebo reference="RFinger12_link">
-        <mu1>0.000002</mu1>
-        <mu2>0.000002</mu2>
-    </gazebo>
-    <gazebo reference="LFinger33_link">
-        <mu1>0.000002</mu1>
-        <mu2>0.000002</mu2>
-    </gazebo>
-    <gazebo reference="RFinger31_link">
-        <mu1>0.000002</mu1>
-        <mu2>0.000002</mu2>
-    </gazebo>
-    <gazebo reference="LFinger21_link">
-        <mu1>0.000002</mu1>
-        <mu2>0.000002</mu2>
-    </gazebo>
-    <gazebo reference="RFinger32_link">
-        <mu1>0.000002</mu1>
-        <mu2>0.000002</mu2>
-    </gazebo>
-    <gazebo reference="LFinger13_link">
-        <mu1>0.000002</mu1>
-        <mu2>0.000002</mu2>
-    </gazebo>
-    <gazebo reference="LFinger32_link">
-        <mu1>0.000002</mu1>
-        <mu2>0.000002</mu2>
-    </gazebo>
-    <gazebo reference="LFinger11_link">
-        <mu1>0.000002</mu1>
-        <mu2>0.000002</mu2>
-    </gazebo>
-    <gazebo reference="RFinger22_link">
-        <mu1>0.000002</mu1>
-        <mu2>0.000002</mu2>
-    </gazebo>
-    <gazebo reference="RFinger13_link">
-        <mu1>0.000002</mu1>
-        <mu2>0.000002</mu2>
-    </gazebo>
-    <gazebo reference="LFinger22_link">
-        <mu1>0.000002</mu1>
-        <mu2>0.000002</mu2>
-    </gazebo>
-    <gazebo reference="RFinger21_link">
-        <mu1>0.000002</mu1>
-        <mu2>0.000002</mu2>
-    </gazebo>
-    <gazebo reference="LFinger41_link">
-        <mu1>0.000002</mu1>
-        <mu2>0.000002</mu2>
-    </gazebo>
-    <gazebo reference="LFinger12_link">
-        <mu1>0.000002</mu1>
-        <mu2>0.000002</mu2>
-    </gazebo>
-    <gazebo reference="RFinger23_link">
-        <mu1>0.000002</mu1>
-        <mu2>0.000002</mu2>
-    </gazebo>
-    <gazebo reference="RFinger11_link">
-        <mu1>0.000002</mu1>
-        <mu2>0.000002</mu2>
-    </gazebo>
-    <gazebo reference="LFinger23_link">
-        <mu1>0.000002</mu1>
-        <mu2>0.000002</mu2>
-    </gazebo>
-    <gazebo reference="LFinger43_link">
-        <mu1>0.000002</mu1>
-        <mu2>0.000002</mu2>
-    </gazebo>
-    <gazebo reference="RFinger43_link">
-        <mu1>0.000002</mu1>
-        <mu2>0.000002</mu2>
-    </gazebo>
-    <gazebo reference="RFinger42_link">
-        <mu1>0.000002</mu1>
-        <mu2>0.000002</mu2>
-    </gazebo>
-    <gazebo reference="LFinger31_link">
-        <mu1>0.000002</mu1>
-        <mu2>0.000002</mu2>
-    </gazebo>
-    <gazebo reference="RFinger33_link">
-        <mu1>0.000002</mu1>
-        <mu2>0.000002</mu2>
-    </gazebo>
-    <gazebo reference="LThumb1_link">
-        <mu1>0.000002</mu1>
-        <mu2>0.000002</mu2>
-    </gazebo>
-    <gazebo reference="RThumb2_link">
-        <mu1>0.000002</mu1>
-        <mu2>0.000002</mu2>
-    </gazebo>
-    <gazebo reference="RThumb1_link">
-        <mu1>0.000002</mu1>
-        <mu2>0.000002</mu2>
-    </gazebo>
-    <gazebo reference="LThumb2_link">
-        <mu1>0.000002</mu1>
-        <mu2>0.000002</mu2>
-    </gazebo>
-    <gazebo reference="WheelFL_link">
-        <mu1>0.000002</mu1>
-        <mu2>0.000002</mu2>
-    </gazebo>
-    <gazebo reference="WheelFR_link">
-        <mu1>0.000002</mu1>
-        <mu2>0.000002</mu2>
-    </gazebo>
-    <gazebo reference="WheelB_link">
-        <mu1>0.000002</mu1>
-        <mu2>0.000002</mu2>
-    </gazebo>
     <!-- Hardware interfaces -->
     <gazebo>
@@ -203,7 +7,209 @@
             <controller_manager_node_name>controller_manager</controller_manager_node_name>
         </plugin>
+    </gazebo>
+    <gazebo>
         <plugin filename="gz-sim-sensors-system" name="gz::sim::systems::Sensors">
             <render_engine>ogre2</render_engine>
         </plugin>
+    </gazebo>
+    <gazebo reference="Neck">
+        <plugin filename="gz-sim-joint-trajectory-system" name="gz::sim::systems::JointTrajectoryController">
+            <topic>/joint_states</topic>
+            <joint_name>HeadYaw</joint_name>
+        </plugin>
+        <mu1>0.2</mu1>
+        <mu2>0.2</mu2>
+    </gazebo>
+    <gazebo reference="Head">
+        <mu1>0.2</mu1>
+        <mu2>0.2</mu2>
+    </gazebo>
+    <gazebo reference="Hip">
+        <mu1>0.2</mu1>
+        <mu2>0.2</mu2>
+    </gazebo>
+    <gazebo reference="Pelvis">
+        <mu1>0.2</mu1>
+        <mu2>0.2</mu2>
+    </gazebo>
+    <gazebo reference="Tibia">
+        <mu1>0.2</mu1>
+        <mu2>0.2</mu2>
+    </gazebo>
+    <gazebo reference="torso">
+        <mu1>0.2</mu1>
+        <mu2>0.2</mu2>
+    </gazebo>
+    <gazebo reference="LShoulder">
+        <mu1>0.2</mu1>
+        <mu2>0.2</mu2>
+    </gazebo>
+    <gazebo reference="LBicep">
+        <mu1>0.2</mu1>
+        <mu2>0.2</mu2>
+    </gazebo>
+    <gazebo reference="LElbow">
+        <mu1>0.2</mu1>
+        <mu2>0.2</mu2>
+    </gazebo>
+    <gazebo reference="LForeArm">
+        <mu1>0.2</mu1>
+        <mu2>0.2</mu2>
+    </gazebo>
+    <gazebo reference="l_wrist">
+        <mu1>0.2</mu1>
+        <mu2>0.2</mu2>
+    </gazebo>
+    <gazebo reference="l_gripper">
+        <mu1>0.2</mu1>
+        <mu2>0.2</mu2>
+    </gazebo>
+    <gazebo reference="RShoulder">
+        <mu1>0.2</mu1>
+        <mu2>0.2</mu2>
+    </gazebo>
+    <gazebo reference="RBicep">
+        <mu1>0.2</mu1>
+        <mu2>0.2</mu2>
+    </gazebo>
+    <gazebo reference="RElbow">
+        <mu1>0.2</mu1>
+        <mu2>0.2</mu2>
+    </gazebo>
+    <gazebo reference="RForeArm">
+        <mu1>0.2</mu1>
+        <mu2>0.2</mu2>
+    </gazebo>
+    <gazebo reference="r_wrist">
+        <mu1>0.2</mu1>
+        <mu2>0.2</mu2>
+    </gazebo>
+    <gazebo reference="r_gripper">
+        <mu1>0.8</mu1>
+        <mu2>0.8</mu2>
+    </gazebo>
+    <gazebo reference="RFinger41_link">
+        <mu1>0.8</mu1>
+        <mu2>0.8</mu2>
+    </gazebo>
+    <gazebo reference="LFinger42_link">
+        <mu1>0.000002</mu1>
+        <mu2>0.000002</mu2>
+    </gazebo>
+    <gazebo reference="RFinger12_link">
+        <mu1>0.000002</mu1>
+        <mu2>0.000002</mu2>
+    </gazebo>
+    <gazebo reference="LFinger33_link">
+        <mu1>0.000002</mu1>
+        <mu2>0.000002</mu2>
+    </gazebo>
+    <gazebo reference="RFinger31_link">
+        <mu1>0.000002</mu1>
+        <mu2>0.000002</mu2>
+    </gazebo>
+    <gazebo reference="LFinger21_link">
+        <mu1>0.000002</mu1>
+        <mu2>0.000002</mu2>
+    </gazebo>
+    <gazebo reference="RFinger32_link">
+        <mu1>0.000002</mu1>
+        <mu2>0.000002</mu2>
+    </gazebo>
+    <gazebo reference="LFinger13_link">
+        <mu1>0.000002</mu1>
+        <mu2>0.000002</mu2>
+    </gazebo>
+    <gazebo reference="LFinger32_link">
+        <mu1>0.000002</mu1>
+        <mu2>0.000002</mu2>
+    </gazebo>
+    <gazebo reference="LFinger11_link">
+        <mu1>0.000002</mu1>
+        <mu2>0.000002</mu2>
+    </gazebo>
+    <gazebo reference="RFinger22_link">
+        <mu1>0.000002</mu1>
+        <mu2>0.000002</mu2>
+    </gazebo>
+    <gazebo reference="RFinger13_link">
+        <mu1>0.000002</mu1>
+        <mu2>0.000002</mu2>
+    </gazebo>
+    <gazebo reference="LFinger22_link">
+        <mu1>0.000002</mu1>
+        <mu2>0.000002</mu2>
+    </gazebo>
+    <gazebo reference="RFinger21_link">
+        <mu1>0.000002</mu1>
+        <mu2>0.000002</mu2>
+    </gazebo>
+    <gazebo reference="LFinger41_link">
+        <mu1>0.000002</mu1>
+        <mu2>0.000002</mu2>
+    </gazebo>
+    <gazebo reference="LFinger12_link">
+        <mu1>0.000002</mu1>
+        <mu2>0.000002</mu2>
+    </gazebo>
+    <gazebo reference="RFinger23_link">
+        <mu1>0.000002</mu1>
+        <mu2>0.000002</mu2>
+    </gazebo>
+    <gazebo reference="RFinger11_link">
+        <mu1>0.000002</mu1>
+        <mu2>0.000002</mu2>
+    </gazebo>
+    <gazebo reference="LFinger23_link">
+        <mu1>0.000002</mu1>
+        <mu2>0.000002</mu2>
+    </gazebo>
+    <gazebo reference="LFinger43_link">
+        <mu1>0.000002</mu1>
+        <mu2>0.000002</mu2>
+    </gazebo>
+    <gazebo reference="RFinger43_link">
+        <mu1>0.000002</mu1>
+        <mu2>0.000002</mu2>
+    </gazebo>
+    <gazebo reference="RFinger42_link">
+        <mu1>0.000002</mu1>
+        <mu2>0.000002</mu2>
+    </gazebo>
+    <gazebo reference="LFinger31_link">
+        <mu1>0.000002</mu1>
+        <mu2>0.000002</mu2>
+    </gazebo>
+    <gazebo reference="RFinger33_link">
+        <mu1>0.000002</mu1>
+        <mu2>0.000002</mu2>
+    </gazebo>
+    <gazebo reference="LThumb1_link">
+        <mu1>0.000002</mu1>
+        <mu2>0.000002</mu2>
+    </gazebo>
+    <gazebo reference="RThumb2_link">
+        <mu1>0.000002</mu1>
+        <mu2>0.000002</mu2>
+    </gazebo>
+    <gazebo reference="RThumb1_link">
+        <mu1>0.000002</mu1>
+        <mu2>0.000002</mu2>
+    </gazebo>
+    <gazebo reference="LThumb2_link">
+        <mu1>0.000002</mu1>
+        <mu2>0.000002</mu2>
+    </gazebo>
+    <gazebo reference="WheelFL_link">
+        <mu1>0.8</mu1>
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