Commit message: Sensors added (not functional at present)

File: hospital_robot_ws/src/hrobot_description/urdf/gazebo_sim_ros2_control.urdf.xacro (robot description, xacro)
@@ -206,3 +206,60 @@
         </plugin>
     </gazebo>
+    <!-- RGBD camera -->
+    <gazebo reference="RGBDCamera_link">
+        <sensor name="rgbd_cam" type="rgbd_camera">
+            <camera>
+                <horizontal_fov>1.5184</horizontal_fov>
+                <image>
+                    <width>424</width>
+                    <height>240</height>
+                </image>
+                <clip>
+                    <near>0.05</near>
+                    <far>1.5</far>
+                </clip>
+            </camera>
+            <always_on>1</always_on>
+            <gz_frame_id>RGBDCamera_link</gz_frame_id>
+            <topic>scan</topic>
+            <update_rate>15.0</update_rate>
+            <visualize>true</visualize>
+        </sensor>
+    </gazebo>
+    <!-- Lidar sensor-->
+    <gazebo reference="LidarSensor_link">
+        <material>
+            <ambient>'0.1 0.1 0.1 1'</ambient>
+            <diffuse>'0.1 0.1 0.1 1'</diffuse>
+            <specular>'0.1 0.1 0.1 1'</specular>
+        </material>
+        <sensor name="lidar_Sensor" type="gpu_lidar">
+            <topic>scan</topic>
+            <update_rate>10</update_rate>
+            <always_on>true</always_on>
+            <visualize>true</visualize>
+            <ray>
+                <scan>
+                    <horizontal>
+                        <samples>720</samples>
+                        <resolution>1</resolution>
+                        <min_angle>-3.14159</min_angle>
+                        <max_angle>3.14159</max_angle>
+                    </horizontal>
+                    <vertical>
+                        <samples>1</samples>
+                        <resolution>1</resolution>
+                        <min_angle>0</min_angle>
+                        <max_angle>0</max_angle>
+                    </vertical>
+                </scan>
+                <range>
+                    <min>0.2</min>
+                    <max>25.0</max>
+                    <resolution>0.225</resolution>
+                </range>
+            </ray>
+            <gz_frame_id>LidarSensor_link</gz_frame_id>
+        </sensor>
+    </gazebo>
 </robot>

File: hospital_robot_ws/src/hrobot_description/urdf/pepper_robot.urdf.xacro (robot description, xacro)
@@ -3,4 +3,8 @@
   <xacro:include filename="$(find hrobot_description)/urdf/gazebo_sim_ros2_control.urdf.xacro" />
   <xacro:include filename="$(find hrobot_description)/urdf/pepper_robot_ros2_control.xacro" />
+  <xacro:include filename="$(find hrobot_description)/urdf/pepper_robot_sensors.xacro" />
+  <material name="light_blue">
+      <color rgba="0.0 0.3 1.0 1.0"/>
+  </material>
   <link name="base_footprint" />
   <link name="base_link"/>
@@ -8,5 +12,5 @@
     <parent link="base_footprint"/>
     <child link="base_link"/>
-    <origin rpy="0 0 0" xyz="0 0 -0.1"/>
+    <origin rpy="0 0 0" xyz="0 0 0"/>
   </joint>
   <joint name="HeadYaw" type="revolute">
@@ -69,4 +73,25 @@
     <limit effort="10.1884" lower="-0.514872" upper="0.514872" velocity="2.27032"/>
   </joint>
+  <xacro:lidar_sensor frame_id="Lidar_Sensor" parent="base_link" xyz_offset="0 0.05 0" rpy_offset="1.57 0 0"/>
+  <xacro:rgbd_camera camera_name="RGBDCamera" parent="Head" xyz_offset="0.105 0 0.12" rpy_offset="0 0.1 0"/>
+  <!-- <link name="Mouth">
+    <visual>
+      <geometry>
+        <box size="0.038 0.04 0.017"/>
+      </geometry>
+      <origin rpy="0 0 0" xyz="0 0 0"/>
+    </visual>
+    <collision>
+      <geometry>
+        <box size="0.01 0.05 0.05"/>
+      </geometry>
+      <origin rpy="0 0 0" xyz="0 0 0"/>
+    </collision>
+  </link>
+  <joint name="Mouth_joint" type="fixed">
+    <parent link="Head"/>
+    <child link="Mouth"/>
+    <origin rpy="0 0.4 0" xyz="0.08 0 0.06"/>
+  </joint> -->
   <link name="Hip">
     <visual>

Commit message: Sensors added (not functional at present)

File: hospital_robot_ws/src/hrobot_description/urdf/gazebo_sim_ros2_control.urdf.xacro (robot description, xacro)
@@ -207,5 +207,5 @@
     </gazebo>
     <!-- RGBD camera -->
-    <gazebo reference="RGBDCamera_link">
+    <gazebo reference="RGBD_Camera_link">
         <sensor name="rgbd_cam" type="rgbd_camera">
             <camera>
@@ -221,12 +221,12 @@
             </camera>
             <always_on>1</always_on>
-            <gz_frame_id>RGBDCamera_link</gz_frame_id>
-            <topic>scan</topic>
+            <gz_frame_id>RGBD_Camera_link</gz_frame_id>
+            <topic>cam</topic>
             <update_rate>15.0</update_rate>
             <visualize>true</visualize>
         </sensor>
     </gazebo>
-    <!-- Lidar sensor-->
-    <gazebo reference="LidarSensor_link">
+    <!-- Lidar sensor -->
+    <gazebo reference="Lidar_Sensor_link">
         <material>
             <ambient>'0.1 0.1 0.1 1'</ambient>
@@ -260,6 +260,21 @@
                 </range>
             </ray>
-            <gz_frame_id>LidarSensor_link</gz_frame_id>
+            <gz_frame_id>Lidar_Sensor_link</gz_frame_id>
         </sensor>
     </gazebo>
+    <!-- IMU sensor -->
+    <gazebo reference="IMU_link">
+        <material>
+            <ambient>'0.1 0.1 0.1 1'</ambient>
+            <diffuse>'0.1 0.1 0.1 1'</diffuse>
+            <specular>'0.1 0.1 0.1 1'</specular>
+        </material>
+        <sensor name="imu_sensor" type="imu">
+            <topic>imu/data</topic>
+            <update_rate>15.0</update_rate>
+            <always_on>true</always_on>
+            <visualize>false</visualize>
+            <gz_frame_id>IMU_link</gz_frame_id>
+        </sensor>
+    </gazebo>
 </robot>

File: hospital_robot_ws/src/hrobot_description/urdf/pepper_robot.urdf.xacro (robot description, xacro)
@@ -73,6 +73,7 @@
     <limit effort="10.1884" lower="-0.514872" upper="0.514872" velocity="2.27032"/>
   </joint>
-  <xacro:lidar_sensor frame_id="Lidar_Sensor" parent="base_link" xyz_offset="0 0.05 0" rpy_offset="1.57 0 0"/>
-  <xacro:rgbd_camera camera_name="RGBDCamera" parent="Head" xyz_offset="0.105 0 0.12" rpy_offset="0 0.1 0"/>
+  <xacro:lidar_sensor frame_id="Lidar_Sensor" parent="base_link" xyz_offset="0 0 0.07" rpy_offset="0 0 0"/>
+  <xacro:rgbd_camera camera_name="RGBD_Camera" parent="Head" xyz_offset="0.105 0 0.12" rpy_offset="0 0.1 0"/>
+  <xacro:imu_sensor frame_id="IMU" parent="base_link" xyz_offset="0 0 0" rpy_offset="0 0 0"/>
   <!-- <link name="Mouth">
     <visual>

File: hospital_robot_ws/src/hrobot_description/urdf/pepper_robot_sensors.xacro (robot description, xacro)
@@ -5,5 +5,5 @@
     <!-- RGBD Camera -->
     <xacro:macro name="rgbd_camera" params="
-        camera_name:='cam_1'
+        camera_name:='RGBD_Camera'
         parent:='base_link'
         mesh_file:='file://$(find hrobot_description)/meshes/sensors/intel_realsense/d435.stl'
@@ -156,5 +156,5 @@
         <link name="${frame_id}">
         <visual>
-            <origin xyz="${mesh_xyz_offset}" rpy="${mesh_rpy_offset}"/>
+            <origin xyz="-0.05 0 -0.029" rpy="1.57 0 0.8"/>
             <geometry>
                 <mesh filename="${mesh_file}" scale="${mesh_scale}"/>
@@ -188,3 +188,55 @@
         </joint>
   </xacro:macro>
+    <!-- IMU sensor -->
+    <xacro:macro name="imu_sensor" params="
+        parent:='base_link'
+        frame_id:='imu'
+        xyz_offset:='0 0 0'
+        rpy_offset:='0 0 0'
+        inertial_xyz_offset:='0 0 0'
+        inertial_rpy_offset:='0 0 0'
+        mass:=0.031
+        length:=0.03899
+        width:=0.03785
+        height:=0.01338
+        material_name:='imu_black'
+        material_color:='0.1 0.1 0.1 1'
+        gazebo_material_ambient:='0.1 0.1 0.1 1'
+        gazebo_material_diffuse:='0.1 0.1 0.1 1'
+        gazebo_material_specular:='0.1 0.1 0.1 1'
+        update_rate:='15.0'
+        topic_name:='imu/data'
+        always_on:=true
+        visualize:=false">
+        <xacro:property name="ixx" value="${(mass/12.0) * (height*height + width*width)}" />
+        <xacro:property name="iyy" value="${(mass/12.0) * (length*length + height*height)}" />
+        <xacro:property name="izz" value="${(mass/12.0) * (length*length + width*width)}" />
+        <link name="${frame_id}_link">
+            <visual>
+                <origin xyz="0 0 0" rpy="0 0 0"/>
+                <geometry>
+                    <box size="${length} ${width} ${height}"/>
+                </geometry>
+                <material name="${material_name}">
+                    <color rgba="${material_color}"/>
+                </material>
+            </visual>
+            <inertial>
+                <mass value="${mass}" />
+                <origin xyz="${inertial_xyz_offset}" rpy="${inertial_rpy_offset}"/>
+                <inertia
+                    ixx="${ixx}"
+                    ixy="0.0"
+                    ixz="0.0"
+                    iyy="${iyy}"
+                    iyz="0.0"
+                    izz="${izz}" />
+            </inertial>
+        </link>
+        <joint name="${frame_id}_joint" type="fixed">
+            <parent link="${parent}"/>
+            <child link="${frame_id}_link" />
+            <origin xyz="${xyz_offset}" rpy="${rpy_offset}"/>
+        </joint>
+    </xacro:macro>
 </robot>

Commit message: Double joint state publishing issue fixed.

File: hospital_robot_ws/src/hrobot_description/urdf/gazebo_sim_ros2_control.urdf.xacro (robot description, xacro)
@@ -206,4 +206,15 @@
         </plugin>
     </gazebo>
+    <!-- Enables navigation
+    <gazebo>
+        <plugin filename="gz-sim-diff-drive-system" name="gz::sim::systems::DiffDrive">
+            <left_joint>WheelFL</left_joint>
+            <right_joint>WheelFR</right_joint>
+            <wheel_separation>0.31</wheel_separation>
+            <wheel_radius>0.08</wheel_radius>
+            <odom_publish_frequency>1</odom_publish_frequency>
+            <topic>cmd_vel</topic>
+        </plugin>
+    </gazebo> -->
     <!-- RGBD camera -->
     <gazebo reference="RGBD_Camera_link">
@@ -229,15 +240,10 @@
     <!-- Lidar sensor -->
     <gazebo reference="Lidar_Sensor_link">
-        <material>
-            <ambient>'0.1 0.1 0.1 1'</ambient>
-            <diffuse>'0.1 0.1 0.1 1'</diffuse>
-            <specular>'0.1 0.1 0.1 1'</specular>
-        </material>
-        <sensor name="lidar_Sensor" type="gpu_lidar">
+        <sensor name="gpu_lidar" type="gpu_lidar">
             <topic>scan</topic>
             <update_rate>10</update_rate>
             <always_on>true</always_on>
             <visualize>true</visualize>
-            <ray>
+            <lidar>
                 <scan>
                     <horizontal>
@@ -249,7 +255,7 @@
                     <vertical>
                         <samples>1</samples>
-                        <resolution>1</resolution>
-                        <min_angle>0</min_angle>
-                        <max_angle>0</max_angle>
+                        <resolution>0.1</resolution>
+                        <min_angle>0.0</min_angle>
+                        <max_angle>0.0</max_angle>
                     </vertical>
                 </scan>
@@ -259,6 +265,6 @@
                     <resolution>0.225</resolution>
                 </range>
-            </ray>
-            <gz_frame_id>Lidar_Sensor_link</gz_frame_id>
+                <frame_id>/Lidar_Sensor_link</frame_id>
+            </lidar>
         </sensor>
     </gazebo>
@@ -273,5 +279,5 @@
             <topic>imu/data</topic>
             <update_rate>15.0</update_rate>
-            <always_on>true</always_on>
+            <always_on>1</always_on>
             <visualize>false</visualize>
             <gz_frame_id>IMU_link</gz_frame_id>

File: hospital_robot_ws/src/hrobot_description/urdf/pepper_robot.urdf.xacro (robot description, xacro)
@@ -1189,9 +1189,9 @@
     </inertial>
   </link>
-  <joint name="WheelB" type="continuous">
+  <joint name="WheelB" type="fixed">
     <parent link="Tibia"/>
     <child link="WheelB_link"/>
     <origin rpy="0 0 0" xyz="-0.17 0 -0.264"/>
-    <axis xyz="0 1 0"/>
+    <!-- <axis xyz="0 1 0"/> -->
   </joint>
 </robot>

File: hospital_robot_ws/src/hrobot_description/urdf/pepper_robot_ros2_control.xacro (robot description, xacro)
@@ -7,13 +7,21 @@
         <!-- Left wheel -->
         <joint name="WheelFL">
-            <command_interface name="velocity"/>
+            <command_interface name="velocity">
+                <param name="min">-1</param>
+                <param name="max">1</param>
+            </command_interface>
             <state_interface name="position"/>
             <state_interface name="velocity"/>
+            <state_interface name="effort"/>
         </joint>
         <!-- Right wheel -->
         <joint name="WheelFR">
-            <command_interface name="velocity"/>
+            <command_interface name="velocity">
+                <param name="min">-1</param>
+                <param name="max">1</param>
+            </command_interface>
             <state_interface name="position"/>
             <state_interface name="velocity"/>
+            <state_interface name="effort"/>
         </joint>
         <!-- Head -->

File: hospital_robot_ws/src/hrobot_description/urdf/pepper_robot_sensors.xacro (robot description, xacro)
@@ -154,38 +154,38 @@
         <xacro:property name="ixx_iyy" value="${(mass/12) * (3 * radius * radius + lidar_height * lidar_height)}" />
         <xacro:property name="izz" value="${(mass/2) * (radius * radius)}" />
-        <link name="${frame_id}">
-        <visual>
-            <origin xyz="-0.05 0 -0.029" rpy="1.57 0 0.8"/>
+        <link name="${frame_id}_link">
+            <visual>
+                <origin xyz="-0.05 0 -0.029" rpy="1.57 0 0.8"/>
+                <geometry>
+                    <mesh filename="${mesh_file}" scale="${mesh_scale}"/>
+                </geometry>
+                <material name="${material_name}">
+                <color rgba="${material_color}"/>
+                </material>
+            </visual>
+            <collision>
+                <origin xyz="${collision_xyz_offset}" rpy="${collision_rpy_offset}"/>
             <geometry>
-                <mesh filename="${mesh_file}" scale="${mesh_scale}"/>
+                <cylinder radius="${lidar_width/2}" length="${lidar_height}"/>
             </geometry>
-            <material name="${material_name}">
-            <color rgba="${material_color}"/>
-            </material>
-        </visual>
-        <collision>
-            <origin xyz="${collision_xyz_offset}" rpy="${collision_rpy_offset}"/>
-        <geometry>
-            <cylinder radius="${lidar_width/2}" length="${lidar_height}"/>
-        </geometry>
-        </collision>
-        <inertial>
-            <mass value="${mass}" />
-            <origin xyz="${inertial_xyz_offset}" rpy="${inertial_rpy_offset}"/>
-            <inertia
-            ixx="${ixx_iyy}"
-            ixy="0.0"
-            ixz="0.0"
-            iyy="${ixx_iyy}"
-            iyz="0.0"
-            izz="${izz}" />
-        </inertial>
+            </collision>
+            <inertial>
+                <mass value="${mass}" />
+                <origin xyz="${inertial_xyz_offset}" rpy="${inertial_rpy_offset}"/>
+                <inertia
+                ixx="${ixx_iyy}"
+                ixy="0.0"
+                ixz="0.0"
+                iyy="${ixx_iyy}"
+                iyz="0.0"
+                izz="${izz}" />
+            </inertial>
         </link>
         <joint name="${frame_id}_joint" type="fixed">
             <parent link="${parent}"/>
-            <child link="${frame_id}" />
+            <child link="${frame_id}_link" />
             <origin xyz="${xyz_offset}" rpy="${rpy_offset}"/>
         </joint>
-  </xacro:macro>
+    </xacro:macro>
     <!-- IMU sensor -->
     <xacro:macro name="imu_sensor" params="

Commit message: Fixed rviz problem for lidar sensor.

File: hospital_robot_ws/src/hrobot_description/urdf/gazebo_sim_ros2_control.urdf.xacro (robot description, xacro)
@@ -218,5 +218,5 @@
     </gazebo> -->
     <!-- RGBD camera -->
-    <gazebo reference="RGBD_Camera_link">
+    <!-- <gazebo reference="RGBD_Camera_link">
         <sensor name="rgbd_cam" type="rgbd_camera">
             <camera>
@@ -237,8 +237,8 @@
             <visualize>true</visualize>
         </sensor>
-    </gazebo>
+    </gazebo> -->
     <!-- Lidar sensor -->
     <gazebo reference="Lidar_Sensor_link">
-        <sensor name="gpu_lidar" type="gpu_lidar">
+        <sensor name="laser_sensor" type="gpu_lidar">
             <topic>scan</topic>
             <update_rate>10</update_rate>
@@ -265,10 +265,10 @@
                     <resolution>0.225</resolution>
                 </range>
-                <frame_id>/Lidar_Sensor_link</frame_id>
             </lidar>
+            <gz_frame_id>Lidar_Sensor_link</gz_frame_id>
         </sensor>
     </gazebo>
     <!-- IMU sensor -->
-    <gazebo reference="IMU_link">
+    <!-- <gazebo reference="IMU_link">
         <material>
             <ambient>'0.1 0.1 0.1 1'</ambient>
@@ -283,4 +283,4 @@
             <gz_frame_id>IMU_link</gz_frame_id>
         </sensor>
-    </gazebo>
+    </gazebo> -->
 </robot>

File: hospital_robot_ws/src/hrobot_description/urdf/pepper_robot_sensors.xacro (robot description, xacro)
@@ -136,5 +136,5 @@
         mass:=0.185
         material_name:='rplidar_black'
-        material_color:='0.1 0.1 0.1 1'
+        material_color:='0.13 0.13 0.13 1.0'
         gazebo_material_ambient:='0.1 0.1 0.1 1'
         gazebo_material_diffuse:='0.1 0.1 0.1 1'
@@ -166,7 +166,7 @@
             <collision>
                 <origin xyz="${collision_xyz_offset}" rpy="${collision_rpy_offset}"/>
-            <geometry>
-                <cylinder radius="${lidar_width/2}" length="${lidar_height}"/>
-            </geometry>
+                <geometry>
+                    <cylinder radius="${lidar_width/2}" length="${lidar_height}"/>
+                </geometry>
             </collision>
             <inertial>
