Commit message: Lidar and rgbd/depth-camera working.

File: hospital_robot_ws/src/hrobot_description/urdf/gazebo_sim_ros2_control.urdf.xacro (robot description, xacro)
@@ -218,5 +218,5 @@
     </gazebo> -->
     <!-- RGBD camera -->
-    <!-- <gazebo reference="RGBD_Camera_link">
+    <gazebo reference="RGBD_Camera_link">
         <sensor name="rgbd_cam" type="rgbd_camera">
             <camera>
@@ -233,9 +233,12 @@
             <always_on>1</always_on>
             <gz_frame_id>RGBD_Camera_link</gz_frame_id>
-            <topic>cam</topic>
+            <topic>cam_1</topic>
             <update_rate>15.0</update_rate>
             <visualize>true</visualize>
         </sensor>
-    </gazebo> -->
+    </gazebo>
+    <gazebo reference="camera_link">
+      <material>Gazebo/Red</material>
+    </gazebo>
     <!-- Lidar sensor -->
     <gazebo reference="Lidar_Sensor_link">
@@ -253,10 +256,17 @@
                         <max_angle>3.14159</max_angle>
                     </horizontal>
+                    <!-- 2D Lidar settings -->
                     <vertical>
                         <samples>1</samples>
-                        <resolution>0.1</resolution>
+                        <resolution>1</resolution>
                         <min_angle>0.0</min_angle>
                         <max_angle>0.0</max_angle>
                     </vertical>
+                    <!-- 3D Lidar settings (PointCloud)-->
+                    <!-- <vertical>
+                        <samples>32</samples>
+                        <min_angle>-0.5353</min_angle>
+                        <max_angle>0.1862</max_angle>
+                    </vertical> -->
                 </scan>
                 <range>

File: hospital_robot_ws/src/hrobot_description/urdf/pepper_robot.urdf.xacro (robot description, xacro)
@@ -74,7 +74,46 @@
   </joint>
   <xacro:lidar_sensor frame_id="Lidar_Sensor" parent="base_link" xyz_offset="0 0 0.07" rpy_offset="0 0 0"/>
-  <xacro:rgbd_camera camera_name="RGBD_Camera" parent="Head" xyz_offset="0.105 0 0.12" rpy_offset="0 0.1 0"/>
-  <xacro:imu_sensor frame_id="IMU" parent="base_link" xyz_offset="0 0 0" rpy_offset="0 0 0"/>
-  <!-- <link name="Mouth">
+  <xacro:rgbd_camera camera_name="RGBD_Camera" parent="base_link" xyz_offset="0.105 0 0.12" rpy_offset="0 0 0"/>
+  <link name='camera_link'>
+    <pose>0 0 0 0 0 0</pose>
+    <visual name='camera_link_visual'>
+      <origin xyz="0.013 0 0.07" rpy="1.57 0 1.57"/>
+      <geometry>
+        <mesh filename="file://$(find hrobot_description)/meshes/sensors/intel_realsense/d435.stl"/>
+      </geometry>
+      <material name="aluminum">
+          <color rgba="0.8 0.8 0.8 1"/>
+      </material>
+    </visual>
+    <collision name='collision'>
+      <origin xyz="0 0 0" rpy="0 0 0"/>
+      <geometry>
+        <box size=".03 .03 .03"/>
+      </geometry>
+    </collision>
+    <inertial>
+      <mass value="0.1"/>
+      <origin xyz="0 0 0" rpy="0 0 0"/>
+      <inertia
+          ixx="1e-6" ixy="0" ixz="0"
+          iyy="1e-6" iyz="0"
+          izz="1e-6"/>
+    </inertial>
+  </link>
+  <joint type="fixed" name="camera_joint">
+    <origin xyz="0.092 0 0.05" rpy="0 0 0"/>
+    <child link="camera_link"/>
+    <parent link="Head"/>
+    <axis xyz="0 1 0" />
+  </joint>
+  <link name="camera_link_optical">
+  </link>
+  <joint type="fixed" name="camera_optical_joint">
+    <origin xyz="0 0 0" rpy="-1.5707 0 -1.5707"/>
+    <child link="camera_link_optical"/>
+    <parent link="camera_link"/>
+  </joint>
+  <!-- <xacro:imu_sensor frame_id="IMU" parent="base_link" xyz_offset="0 0 0" rpy_offset="0 0 0"/> -->
+  <link name="Mouth">
     <visual>
       <geometry>
@@ -94,5 +133,5 @@
     <child link="Mouth"/>
     <origin rpy="0 0.4 0" xyz="0.08 0 0.06"/>
-  </joint> -->
+  </joint>
   <link name="Hip">
     <visual>

File: hospital_robot_ws/src/hrobot_description/urdf/pepper_robot_sensors.xacro (robot description, xacro)
@@ -3,7 +3,7 @@
     <!-- Source: https://github.com/automaticaddison/yahboom_rosmaster/tree/main/yahboom_rosmaster_description/urdf/sensors -->
     <xacro:property name="M_PI" value="3.1415926535897931" />
-    <!-- RGBD Camera -->
+    <!-- RGBD camera -->
     <xacro:macro name="rgbd_camera" params="
-        camera_name:='RGBD_Camera'
+        camera_name:='rgbd_camera'
         parent:='base_link'
         mesh_file:='file://$(find hrobot_description)/meshes/sensors/intel_realsense/d435.stl'
@@ -37,6 +37,12 @@
         izz:=0.003879257
         material_name:='aluminum'
-        material_color:='0.5 0.5 0.5 1'
+        material_color:='0.8 0.8 0.8 1'
+        horizontal_fov:=1.5184
+        image_width:=424
+        image_height:=240
+        clip_near:=0.05
+        clip_far:=1.5
         update_rate:=2
+        always_on:=1
         visualize:=true
         enable_collision:=false">
@@ -45,8 +51,9 @@
                 <origin xyz="${mesh_xyz_offset}" rpy="${mesh_rpy_offset}"/>
                 <geometry>
-                    <mesh filename="${mesh_file}" />
+                    <!-- <mesh filename="${mesh_file}" /> -->
+                    <box size=".03 .03 .03"/>
                 </geometry>
                 <material name="${material_name}">
-                <color rgba="${material_color}"/>
+                    <color rgba="${material_color}"/>
                 </material>
             </visual>
@@ -189,5 +196,5 @@
     </xacro:macro>
     <!-- IMU sensor -->
-    <xacro:macro name="imu_sensor" params="
+    <!-- <xacro:macro name="imu_sensor" params="
         parent:='base_link'
         frame_id:='imu'
@@ -239,4 +246,4 @@
             <origin xyz="${xyz_offset}" rpy="${rpy_offset}"/>
         </joint>
-    </xacro:macro>
+    </xacro:macro> -->
 </robot>
