Commit message: world choosing at startup implemented (only world name needed without extension)

File: hospital_robot_ws/src/hrobot_description/urdf/pepper_robot.urdf.xacro (robot description, xacro)
@@ -1228,9 +1228,10 @@
     </inertial>
   </link>
-  <joint name="WheelB" type="fixed">
+  <joint name="WheelB" type="continuous">
     <parent link="Tibia"/>
     <child link="WheelB_link"/>
     <origin rpy="0 0 0" xyz="-0.17 0 -0.264"/>
-    <!-- <axis xyz="0 1 0"/> -->
+    <dynamics damping="0.0001" friction="0.0"/>
+    <limit effort="0.0" velocity="100.0"/>
   </joint>
 </robot>

File: hospital_robot_ws/src/hrobot_description/urdf/pepper_robot_gazebo.xacro (robot description, xacro)
@@ -186,16 +186,21 @@
     </gazebo>
     <gazebo reference="WheelFL_link">
-        <mu1>0.8</mu1>
-        <mu2>0.8</mu2>
+        <mu1>0.0001</mu1>
+        <mu2>0.0001</mu2>
+        <kp>1000</kp>
+        <kd>10</kd>
     </gazebo>
     <gazebo reference="WheelFR_link">
-        <mu1>0.8</mu1>
-        <mu2>0.8</mu2>
+        <mu1>0.0001</mu1>
+        <mu2>0.0001</mu2>
+        <kp>1000</kp>
+        <kd>10</kd>
     </gazebo>
     <gazebo reference="WheelB_link">
-        <mu1>0.5</mu1>
-        <mu2>0.5</mu2>
-        <kp>1000000</kp>
-        <kd>1000</kd>
+        <!-- Friction parameters: set to near zero -->
+        <mu1>0.0001</mu1>
+        <mu2>0.0001</mu2>
+        <kp>1000</kp>   <!-- lower contact stiffness -->
+        <kd>10</kd>   <!-- lower contact damping -->
     </gazebo>
     <!-- Enables the communication with ros2_control -->
