Commit message: All packages refactored (packages names changed to hospibot_*)

File: hospibot_ws/src/hospibot_description/urdf/hospibot.urdf.xacro (robot description, xacro)
@@ -1,7 +1,7 @@
 <?xml version="1.0"?>
-<robot name="pepper_robot" xmlns:xacro="http://www.ros.org/wiki/xacro">
-  <xacro:include filename="$(find hrobot_description)/urdf/pepper_robot_gazebo.xacro" />
-  <xacro:include filename="$(find hrobot_description)/urdf/pepper_robot_control.xacro" />
-  <xacro:include filename="$(find hrobot_description)/urdf/pepper_robot_sensors.xacro" />
+<robot name="hospibot" xmlns:xacro="http://www.ros.org/wiki/xacro">
+  <xacro:include filename="$(find hospibot_description)/urdf/hospibot_gazebo.xacro" />
+  <xacro:include filename="$(find hospibot_description)/urdf/hospibot_control.xacro" />
+  <xacro:include filename="$(find hospibot_description)/urdf/hospibot_sensors.xacro" />
   <material name="light_blue">
       <color rgba="0.0 0.3 1.0 1.0"/>
@@ -24,11 +24,11 @@
     <visual>
       <geometry>
-        <mesh filename="file://$(find hrobot_description)/meshes/HeadYaw.dae" scale="0.1 0.1 0.1"/>
-      </geometry>
-      <origin rpy="0 0 0" xyz="0 0 0"/>
-    </visual>
-    <collision>
-      <geometry>
-        <mesh filename="file://$(find hrobot_description)/meshes/HeadYaw_0.10.stl" scale="0.1 0.1 0.1"/>
+        <mesh filename="file://$(find hospibot_description)/meshes/HeadYaw.dae" scale="0.1 0.1 0.1"/>
+      </geometry>
+      <origin rpy="0 0 0" xyz="0 0 0"/>
+    </visual>
+    <collision>
+      <geometry>
+        <mesh filename="file://$(find hospibot_description)/meshes/HeadYaw_0.10.stl" scale="0.1 0.1 0.1"/>
       </geometry>
       <origin rpy="0 0 0" xyz="0 0 0"/>
@@ -50,11 +50,11 @@
     <visual>
       <geometry>
-        <mesh filename="file://$(find hrobot_description)/meshes/HeadPitch.dae" scale="0.1 0.1 0.1"/>
-      </geometry>
-      <origin rpy="0 0 0" xyz="0 0 0"/>
-    </visual>
-    <collision>
-      <geometry>
-        <mesh filename="file://$(find hrobot_description)/meshes/HeadPitch_0.10.stl" scale="0.1 0.1 0.1"/>
+        <mesh filename="file://$(find hospibot_description)/meshes/HeadPitch.dae" scale="0.1 0.1 0.1"/>
+      </geometry>
+      <origin rpy="0 0 0" xyz="0 0 0"/>
+    </visual>
+    <collision>
+      <geometry>
+        <mesh filename="file://$(find hospibot_description)/meshes/HeadPitch_0.10.stl" scale="0.1 0.1 0.1"/>
       </geometry>
       <origin rpy="0 0 0" xyz="0 0 0"/>
@@ -80,5 +80,5 @@
       <origin xyz="0.013 0 0.07" rpy="1.57 0 1.57"/>
       <geometry>
-        <mesh filename="file://$(find hrobot_description)/meshes/sensors/intel_realsense/d435.stl"/>
+        <mesh filename="file://$(find hospibot_description)/meshes/sensors/intel_realsense/d435.stl"/>
       </geometry>
       <material name="aluminum">
@@ -137,5 +137,5 @@
     <visual>
       <geometry>
-        <mesh filename="file://$(find hrobot_description)/meshes/HipRoll.dae" scale="0.1 0.1 0.1"/>
+        <mesh filename="file://$(find hospibot_description)/meshes/HipRoll.dae" scale="0.1 0.1 0.1"/>
       </geometry>
       <origin rpy="0 0 0" xyz="0 0 0.079"/>
@@ -143,5 +143,5 @@
     <collision>
       <geometry>
-        <mesh filename="file://$(find hrobot_description)/meshes/HipRoll_0.10.stl" scale="0.1 0.1 0.1"/>
+        <mesh filename="file://$(find hospibot_description)/meshes/HipRoll_0.10.stl" scale="0.1 0.1 0.1"/>
       </geometry>
       <origin rpy="0 0 0" xyz="0 0 0.079"/>
@@ -163,5 +163,5 @@
     <visual>
       <geometry>
-        <mesh filename="file://$(find hrobot_description)/meshes/HipPitch.dae" scale="0.1 0.1 0.1"/>
+        <mesh filename="file://$(find hospibot_description)/meshes/HipPitch.dae" scale="0.1 0.1 0.1"/>
       </geometry>
       <origin rpy="0 0 0" xyz="0 0 0.268"/>
@@ -169,5 +169,5 @@
     <collision>
       <geometry>
-        <mesh filename="file://$(find hrobot_description)/meshes/HipPitch_0.10.stl" scale="0.1 0.1 0.1"/>
+        <mesh filename="file://$(find hospibot_description)/meshes/HipPitch_0.10.stl" scale="0.1 0.1 0.1"/>
       </geometry>
       <origin rpy="0 0 0" xyz="0 0 0.268"/>
@@ -189,11 +189,11 @@
     <visual>
       <geometry>
-        <mesh filename="file://$(find hrobot_description)/meshes/KneePitch.dae" scale="0.1 0.1 0.1"/>
-      </geometry>
-      <origin rpy="0 0 0" xyz="0 0 0"/>
-    </visual>
-    <collision>
-      <geometry>
-        <mesh filename="file://$(find hrobot_description)/meshes/KneePitch_0.10.stl" scale="0.1 0.1 0.1"/>
+        <mesh filename="file://$(find hospibot_description)/meshes/KneePitch.dae" scale="0.1 0.1 0.1"/>
+      </geometry>
+      <origin rpy="0 0 0" xyz="0 0 0"/>
+    </visual>
+    <collision>
+      <geometry>
+        <mesh filename="file://$(find hospibot_description)/meshes/KneePitch_0.10.stl" scale="0.1 0.1 0.1"/>
       </geometry>
       <origin rpy="0 0 0" xyz="0 0 0"/>
@@ -213,5 +213,5 @@
     <visual>
       <geometry>
-        <mesh filename="file://$(find hrobot_description)/meshes/Torso.dae" scale="0.1 0.1 0.1"/>
+        <mesh filename="file://$(find hospibot_description)/meshes/Torso.dae" scale="0.1 0.1 0.1"/>
       </geometry>
       <origin rpy="0 0 0" xyz="2e-05 0 0.139"/>
@@ -219,5 +219,5 @@
     <collision>
       <geometry>
-        <mesh filename="file://$(find hrobot_description)/meshes/Torso_0.10.stl" scale="0.1 0.1 0.1"/>
+        <mesh filename="file://$(find hospibot_description)/meshes/Torso_0.10.stl" scale="0.1 0.1 0.1"/>
       </geometry>
       <origin rpy="0 0 0" xyz="2e-05 0 0.139"/>
@@ -239,11 +239,11 @@
     <visual>
       <geometry>
-        <mesh filename="file://$(find hrobot_description)/meshes/LShoulderPitch.dae" scale="0.1 0.1 0.1"/>
-      </geometry>
-      <origin rpy="0 0 0" xyz="0 0 0"/>
-    </visual>
-    <collision>
-      <geometry>
-        <mesh filename="file://$(find hrobot_description)/meshes/LShoulderPitch_0.10.stl" scale="0.1 0.1 0.1"/>
+        <mesh filename="file://$(find hospibot_description)/meshes/LShoulderPitch.dae" scale="0.1 0.1 0.1"/>
+      </geometry>
+      <origin rpy="0 0 0" xyz="0 0 0"/>
+    </visual>
+    <collision>
+      <geometry>
+        <mesh filename="file://$(find hospibot_description)/meshes/LShoulderPitch_0.10.stl" scale="0.1 0.1 0.1"/>
       </geometry>
       <origin rpy="0 0 0" xyz="0 0 0"/>
@@ -265,11 +265,11 @@
     <visual>
       <geometry>
-        <mesh filename="file://$(find hrobot_description)/meshes/LShoulderRoll.dae" scale="0.1 0.1 0.1"/>
-      </geometry>
-      <origin rpy="0 0 0" xyz="0 0 0"/>
-    </visual>
-    <collision>
-      <geometry>
-        <mesh filename="file://$(find hrobot_description)/meshes/LShoulderRoll_0.10.stl" scale="0.1 0.1 0.1"/>
+        <mesh filename="file://$(find hospibot_description)/meshes/LShoulderRoll.dae" scale="0.1 0.1 0.1"/>
+      </geometry>
+      <origin rpy="0 0 0" xyz="0 0 0"/>
+    </visual>
+    <collision>
+      <geometry>
+        <mesh filename="file://$(find hospibot_description)/meshes/LShoulderRoll_0.10.stl" scale="0.1 0.1 0.1"/>
       </geometry>
       <origin rpy="0 0 0" xyz="0 0 0"/>
@@ -291,11 +291,11 @@
     <visual>
       <geometry>
-        <mesh filename="file://$(find hrobot_description)/meshes/LElbowYaw.dae" scale="0.1 0.1 0.1"/>
-      </geometry>
-      <origin rpy="0 0 0" xyz="0 0 0"/>
-    </visual>
-    <collision>
-      <geometry>
-        <mesh filename="file://$(find hrobot_description)/meshes/LElbowYaw_0.10.stl" scale="0.1 0.1 0.1"/>
+        <mesh filename="file://$(find hospibot_description)/meshes/LElbowYaw.dae" scale="0.1 0.1 0.1"/>
+      </geometry>
+      <origin rpy="0 0 0" xyz="0 0 0"/>
+    </visual>
+    <collision>
+      <geometry>
+        <mesh filename="file://$(find hospibot_description)/meshes/LElbowYaw_0.10.stl" scale="0.1 0.1 0.1"/>
       </geometry>
       <origin rpy="0 0 0" xyz="0 0 0"/>
@@ -317,11 +317,11 @@
     <visual>
       <geometry>
-        <mesh filename="file://$(find hrobot_description)/meshes/LElbowRoll.dae" scale="0.1 0.1 0.1"/>
-      </geometry>
-      <origin rpy="0 0 0" xyz="0 0 0"/>
-    </visual>
-    <collision>
-      <geometry>
-        <mesh filename="file://$(find hrobot_description)/meshes/LElbowRoll_0.10.stl" scale="0.1 0.1 0.1"/>
+        <mesh filename="file://$(find hospibot_description)/meshes/LElbowRoll.dae" scale="0.1 0.1 0.1"/>
+      </geometry>
+      <origin rpy="0 0 0" xyz="0 0 0"/>
+    </visual>
+    <collision>
+      <geometry>
+        <mesh filename="file://$(find hospibot_description)/meshes/LElbowRoll_0.10.stl" scale="0.1 0.1 0.1"/>
       </geometry>
       <origin rpy="0 0 0" xyz="0 0 0"/>
@@ -343,11 +343,11 @@
     <visual>
       <geometry>
-        <mesh filename="file://$(find hrobot_description)/meshes/LWristYaw.dae" scale="0.1 0.1 0.1"/>
-      </geometry>
-      <origin rpy="0 0 0" xyz="0 0 0"/>
-    </visual>
-    <collision>
-      <geometry>
-        <mesh filename="file://$(find hrobot_description)/meshes/LWristYaw_0.10.stl" scale="0.1 0.1 0.1"/>
+        <mesh filename="file://$(find hospibot_description)/meshes/LWristYaw.dae" scale="0.1 0.1 0.1"/>
+      </geometry>
+      <origin rpy="0 0 0" xyz="0 0 0"/>
+    </visual>
+    <collision>
+      <geometry>
+        <mesh filename="file://$(find hospibot_description)/meshes/LWristYaw_0.10.stl" scale="0.1 0.1 0.1"/>
       </geometry>
       <origin rpy="0 0 0" xyz="0 0 0"/>
@@ -382,11 +382,11 @@
     <visual>
       <geometry>
-        <mesh filename="file://$(find hrobot_description)/meshes/RShoulderPitch.dae" scale="0.1 0.1 0.1"/>
-      </geometry>
-      <origin rpy="0 0 0" xyz="0 0 0"/>
-    </visual>
-    <collision>
-      <geometry>
-        <mesh filename="file://$(find hrobot_description)/meshes/RShoulderPitch_0.10.stl" scale="0.1 0.1 0.1"/>
+        <mesh filename="file://$(find hospibot_description)/meshes/RShoulderPitch.dae" scale="0.1 0.1 0.1"/>
+      </geometry>
+      <origin rpy="0 0 0" xyz="0 0 0"/>
+    </visual>
+    <collision>
+      <geometry>
+        <mesh filename="file://$(find hospibot_description)/meshes/RShoulderPitch_0.10.stl" scale="0.1 0.1 0.1"/>
       </geometry>
       <origin rpy="0 0 0" xyz="0 0 0"/>
@@ -408,11 +408,11 @@
     <visual>
       <geometry>
-        <mesh filename="file://$(find hrobot_description)/meshes/RShoulderRoll.dae" scale="0.1 0.1 0.1"/>
-      </geometry>
-      <origin rpy="0 0 0" xyz="0 0 0"/>
-    </visual>
-    <collision>
-      <geometry>
-        <mesh filename="file://$(find hrobot_description)/meshes/RShoulderRoll_0.10.stl" scale="0.1 0.1 0.1"/>
+        <mesh filename="file://$(find hospibot_description)/meshes/RShoulderRoll.dae" scale="0.1 0.1 0.1"/>
+      </geometry>
+      <origin rpy="0 0 0" xyz="0 0 0"/>
+    </visual>
+    <collision>
+      <geometry>
+        <mesh filename="file://$(find hospibot_description)/meshes/RShoulderRoll_0.10.stl" scale="0.1 0.1 0.1"/>
       </geometry>
       <origin rpy="0 0 0" xyz="0 0 0"/>
@@ -434,11 +434,11 @@
     <visual>
       <geometry>
-        <mesh filename="file://$(find hrobot_description)/meshes/RElbowYaw.dae" scale="0.1 0.1 0.1"/>
-      </geometry>
-      <origin rpy="0 0 0" xyz="0 0 0"/>
-    </visual>
-    <collision>
-      <geometry>
-        <mesh filename="file://$(find hrobot_description)/meshes/RElbowYaw_0.10.stl" scale="0.1 0.1 0.1"/>
+        <mesh filename="file://$(find hospibot_description)/meshes/RElbowYaw.dae" scale="0.1 0.1 0.1"/>
+      </geometry>
+      <origin rpy="0 0 0" xyz="0 0 0"/>
+    </visual>
+    <collision>
+      <geometry>
+        <mesh filename="file://$(find hospibot_description)/meshes/RElbowYaw_0.10.stl" scale="0.1 0.1 0.1"/>
       </geometry>
       <origin rpy="0 0 0" xyz="0 0 0"/>
@@ -460,11 +460,11 @@
     <visual>
       <geometry>
-        <mesh filename="file://$(find hrobot_description)/meshes/RElbowRoll.dae" scale="0.1 0.1 0.1"/>
-      </geometry>
-      <origin rpy="0 0 0" xyz="0 0 0"/>
-    </visual>
-    <collision>
-      <geometry>
-        <mesh filename="file://$(find hrobot_description)/meshes/RElbowRoll_0.10.stl" scale="0.1 0.1 0.1"/>
+        <mesh filename="file://$(find hospibot_description)/meshes/RElbowRoll.dae" scale="0.1 0.1 0.1"/>
+      </geometry>
+      <origin rpy="0 0 0" xyz="0 0 0"/>
+    </visual>
+    <collision>
+      <geometry>
+        <mesh filename="file://$(find hospibot_description)/meshes/RElbowRoll_0.10.stl" scale="0.1 0.1 0.1"/>
       </geometry>
       <origin rpy="0 0 0" xyz="0 0 0"/>
@@ -486,11 +486,11 @@
     <visual>
       <geometry>
-        <mesh filename="file://$(find hrobot_description)/meshes/RWristYaw.dae" scale="0.1 0.1 0.1"/>
-      </geometry>
-      <origin rpy="0 0 0" xyz="0 0 0"/>
-    </visual>
-    <collision>
-      <geometry>
-        <mesh filename="file://$(find hrobot_description)/meshes/RWristYaw_0.10.stl" scale="0.1 0.1 0.1"/>
+        <mesh filename="file://$(find hospibot_description)/meshes/RWristYaw.dae" scale="0.1 0.1 0.1"/>
+      </geometry>
+      <origin rpy="0 0 0" xyz="0 0 0"/>
+    </visual>
+    <collision>
+      <geometry>
+        <mesh filename="file://$(find hospibot_description)/meshes/RWristYaw_0.10.stl" scale="0.1 0.1 0.1"/>
       </geometry>
       <origin rpy="0 0 0" xyz="0 0 0"/>
@@ -518,11 +518,11 @@
     <visual>
       <geometry>
-        <mesh filename="file://$(find hrobot_description)/meshes/RFinger41.dae" scale="0.1 0.1 0.1"/>
-      </geometry>
-      <origin rpy="0 0 0" xyz="0 0 0"/>
-    </visual>
-    <collision>
-      <geometry>
-        <mesh filename="file://$(find hrobot_description)/meshes/RFinger41_0.10.stl" scale="0.1 0.1 0.1"/>
+        <mesh filename="file://$(find hospibot_description)/meshes/RFinger41.dae" scale="0.1 0.1 0.1"/>
+      </geometry>
+      <origin rpy="0 0 0" xyz="0 0 0"/>
+    </visual>
+    <collision>
+      <geometry>
+        <mesh filename="file://$(find hospibot_description)/meshes/RFinger41_0.10.stl" scale="0.1 0.1 0.1"/>
       </geometry>
       <origin rpy="0 0 0" xyz="0 0 0"/>
@@ -541,11 +541,11 @@
     <visual>
       <geometry>
-        <mesh filename="file://$(find hrobot_description)/meshes/LFinger42.dae" scale="0.1 0.1 0.1"/>
-      </geometry>
-      <origin rpy="0 0 0" xyz="0 0 0"/>
-    </visual>
-    <collision>
-      <geometry>
-        <mesh filename="file://$(find hrobot_description)/meshes/LFinger42_0.10.stl" scale="0.1 0.1 0.1"/>
+        <mesh filename="file://$(find hospibot_description)/meshes/LFinger42.dae" scale="0.1 0.1 0.1"/>
+      </geometry>
+      <origin rpy="0 0 0" xyz="0 0 0"/>
+    </visual>
+    <collision>
+      <geometry>
+        <mesh filename="file://$(find hospibot_description)/meshes/LFinger42_0.10.stl" scale="0.1 0.1 0.1"/>
       </geometry>
       <origin rpy="0 0 0" xyz="0 0 0"/>
@@ -564,11 +564,11 @@
     <visual>
       <geometry>
-        <mesh filename="file://$(find hrobot_description)/meshes/RFinger12.dae" scale="0.1 0.1 0.1"/>
-      </geometry>
-      <origin rpy="0 0 0" xyz="0 0 0"/>
-    </visual>
-    <collision>
-      <geometry>
-        <mesh filename="file://$(find hrobot_description)/meshes/RFinger12_0.10.stl" scale="0.1 0.1 0.1"/>
+        <mesh filename="file://$(find hospibot_description)/meshes/RFinger12.dae" scale="0.1 0.1 0.1"/>
+      </geometry>
+      <origin rpy="0 0 0" xyz="0 0 0"/>
+    </visual>
+    <collision>
+      <geometry>
+        <mesh filename="file://$(find hospibot_description)/meshes/RFinger12_0.10.stl" scale="0.1 0.1 0.1"/>
       </geometry>
       <origin rpy="0 0 0" xyz="0 0 0"/>
@@ -587,11 +587,11 @@
     <visual>
       <geometry>
-        <mesh filename="file://$(find hrobot_description)/meshes/LFinger33.dae" scale="0.1 0.1 0.1"/>
-      </geometry>
-      <origin rpy="0 0 0" xyz="0 0 0"/>
-    </visual>
-    <collision>
-      <geometry>
-        <mesh filename="file://$(find hrobot_description)/meshes/LFinger33_0.10.stl" scale="0.1 0.1 0.1"/>
+        <mesh filename="file://$(find hospibot_description)/meshes/LFinger33.dae" scale="0.1 0.1 0.1"/>
+      </geometry>
+      <origin rpy="0 0 0" xyz="0 0 0"/>
+    </visual>
+    <collision>
+      <geometry>
+        <mesh filename="file://$(find hospibot_description)/meshes/LFinger33_0.10.stl" scale="0.1 0.1 0.1"/>
       </geometry>
       <origin rpy="0 0 0" xyz="0 0 0"/>
@@ -610,11 +610,11 @@
     <visual>
       <geometry>
-        <mesh filename="file://$(find hrobot_description)/meshes/RFinger31.dae" scale="0.1 0.1 0.1"/>
-      </geometry>
-      <origin rpy="0 0 0" xyz="0 0 0"/>
-    </visual>
-    <collision>
-      <geometry>
-        <mesh filename="file://$(find hrobot_description)/meshes/RFinger31_0.10.stl" scale="0.1 0.1 0.1"/>
+        <mesh filename="file://$(find hospibot_description)/meshes/RFinger31.dae" scale="0.1 0.1 0.1"/>
+      </geometry>
+      <origin rpy="0 0 0" xyz="0 0 0"/>
+    </visual>
+    <collision>
+      <geometry>
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
File: hospibot_ws/src/hospibot_description/urdf/hospibot_control.xacro (robot description, xacro)
@@ -1,5 +1,5 @@
 <?xml version="1.0"?>
-<robot name="pepper_robot" xmlns:xacro="http://www.ros.org/wiki/xacro">
-    <ros2_control name="hospital_robot_hardware_interface" type="system">
+<robot name="hospibot" xmlns:xacro="http://www.ros.org/wiki/xacro">
+    <ros2_control name="hospibot_hardware_interface" type="system">
         <hardware>
             <plugin>gz_ros2_control/GazeboSimSystem</plugin>

File: hospibot_ws/src/hospibot_description/urdf/hospibot_gazebo.xacro (robot description, xacro)
@@ -207,5 +207,5 @@
     <gazebo>
         <plugin name="gz_ros2_control::GazeboSimROS2ControlPlugin" filename="libgz_ros2_control-system.so">
-            <parameters>$(find hrobot_bringup)/config/controllers.yaml</parameters>
+            <parameters>$(find hospibot_bringup)/config/controllers.yaml</parameters>
             <controller_manager_node_name>controller_manager</controller_manager_node_name>
         </plugin>

File: hospibot_ws/src/hospibot_description/urdf/hospibot_sensors.xacro (robot description, xacro)
@@ -7,5 +7,5 @@
         camera_name:='rgbd_camera'
         parent:='base_link'
-        mesh_file:='file://$(find hrobot_description)/meshes/sensors/intel_realsense/d435.stl'
+        mesh_file:='file://$(find hospibot_description)/meshes/sensors/intel_realsense/d435.stl'
         xyz_offset:='0.105 0 0.05'
         rpy_offset:='0 -0.50 0'
@@ -129,5 +129,5 @@
         parent:='base_link'
         frame_id:='laser_frame'
-        mesh_file:='file://$(find hrobot_description)/meshes/sensors/rplidar/RPLIDAR_A3.STL'
+        mesh_file:='file://$(find hospibot_description)/meshes/sensors/rplidar/RPLIDAR_A3.STL'
         xyz_offset:='0 0 0.0825'
         rpy_offset:='0 0 0'
